File: acoustic-carrier-hw/acoustic-carrier-board/processing.kicad_sch (KiCad schematic)
At the start: 25 parts, among them IC1 ECP5-BGA256, J2 Conn_01x04_Socket, J4 Conn_01x06_Socket, J5 Conn_01x02_Socket, U4 W25Q128JVS, U9 W25Q128JVS

Commit message: [carrier] Fixed most of the carrier board ERC issues (next) fix BGA ERC issue
Parts:
- IC1: footprint BGA256C80P16X16_1400X1400X170 -> fpga:BGA256C80P16X16_1400X1400X170; LPN (none) -> C1521614; MPN (none) -> LFE5U-25F-6BG256C; Part Number LFE5U-12F-6BG256C -> LFE5U-25F-6BG256C
Connections:
- net FPGA_USB_RTSn: now reaches IC1.T6 (D7/PB4A)
- net Vcc_IO8 renamed VCORE_3V3
- no-connect marks 8 -> 7
Other:
- note removed: "Vcc_IO8"
Changed lines of the file:
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@@
 		)
 	)
-	(text "Vcc_IO8"
-		(exclude_from_sim no)
-		(at 36.83 21.59 0)
-		(effects
-			(font
-				(size 1.27 1.27)
-			)
-		)
-	)
 	(text "Pure signaling function\nFPGA_DONE: Startup sequence in prograss\nFPGA_INITn: Ready to be configured\nFPGRA_RESET: Initiates configuration sequence when asserted low"
 		(exclude_from_sim no)
@@
 	(text "pullups for Master SPI (MSPI) required by\nTN1260: lattice ECP5 sysCONFIG guide section 6"
 		(exclude_from_sim no)
-		(at 214.884 117.348 0)
+		(at 218.186 113.792 0)
 		(effects
 			(font
@@
 	)
 	(junction
+		(at 251.46 121.92)
+		(diameter 0)
+		(color 0 0 0 0)
+	)
+	(junction
 		(at 177.8 120.65)
 		(diameter 0)
@@
 		(color 0 0 0 0)
 	)
+	(junction
+		(at 190.5 120.65)
+		(diameter 0)
+		(color 0 0 0 0)
+	)
 	(no_connect
 		(at 57.15 59.69)
@@
 	)
 	(no_connect
-		(at 57.15 29.21)
-	)
-	(no_connect
 		(at 57.15 52.07)
 	)
@@
 	(wire
 		(pts
-			(xy 181.61 120.65) (xy 181.61 116.84)
-		)
-		(stroke
-			(width 0)
-			(type default)
-		)
-	)
-	(wire
-		(pts
 			(xy 166.37 127) (xy 166.37 139.7)
 		)
@@
 	(wire
 		(pts
-			(xy 236.22 119.38) (xy 236.22 124.46)
+			(xy 236.22 121.92) (xy 236.22 124.46)
 		)
 		(stroke
@@
 	(wire
 		(pts
-			(xy 26.67 21.59) (xy 31.75 21.59)
+			(xy 26.67 21.59) (xy 27.94 21.59)
 		)
 		(stroke
@@
 	(wire
 		(pts
-			(xy 255.27 58.42) (xy 240.03 58.42)
+			(xy 252.73 58.42) (xy 240.03 58.42)
 		)
 		(stroke
@@
 	(wire
 		(pts
-			(xy 198.12 121.92) (xy 190.5 121.92)
-		)
-		(stroke
-			(width 0)
-			(type default)
-		)
-	)
-	(wire
-		(pts
 			(xy 156.21 144.78) (xy 158.75 144.78)
 		)
@@
 	(wire
 		(pts
-			(xy 190.5 121.92) (xy 190.5 127)
+			(xy 190.5 120.65) (xy 190.5 127)
 		)
 		(stroke
@@
 	(wire
 		(pts
-			(xy 181.61 120.65) (xy 177.8 120.65)
+			(xy 177.8 120.65) (xy 190.5 120.65)
 		)
 		(stroke
@@
 	(wire
 		(pts
-			(xy 255.27 85.09) (xy 248.92 85.09)
+			(xy 252.73 85.09) (xy 248.92 85.09)
 		)
 		(stroke
@@
 	(wire
 		(pts
-			(xy 241.3 119.38) (xy 236.22 119.38)
+			(xy 236.22 121.92) (xy 251.46 121.92)
 		)
 		(stroke
@@
 	(wire
 		(pts
+			(xy 190.5 120.65) (xy 198.12 120.65)
+		)
+		(stroke
+			(width 0)
+			(type default)
+		)
+	)
+	(wire
+		(pts
 			(xy 166.37 120.65) (xy 170.18 120.65)
 		)
@@
 	(wire
 		(pts
+			(xy 57.15 29.21) (xy 62.23 29.21)
+		)
+		(stroke
+			(width 0)
+			(type default)
+		)
+	)
+	(wire
+		(pts
 			(xy 259.08 121.92) (xy 251.46 121.92)
 		)
@@
 		)
 	)
-	(global_label "Vcc_IO8"
+	(global_label "VCORE_3V3"
 		(shape passive)
-		(at 181.61 116.84 0)
+		(at 219.71 26.67 180)
 		(fields_autoplaced yes)
 		(effects
@@
 				(size 1.27 1.27)
 			)
-			(justify left)
+			(justify right)
 		)
 		(property "Intersheetrefs" "${INTERSHEET_REFS}"
-			(at 190.8621 116.84 0)
+			(at 207.2528 26.67 0)
 			(effects
 				(font
 					(size 1.27 1.27)
 				)
-				(justify left)
+				(justify right)
 				(hide yes)
 			)
 		)
 	)
-	(global_label "Vcc_IO8"
+	(global_label "VCORE_3V3"
 		(shape passive)
-		(at 259.08 121.92 0)
+		(at 27.94 21.59 0)
 		(fields_autoplaced yes)
 		(effects
@@
 		)
 		(property "Intersheetrefs" "${INTERSHEET_REFS}"
-			(at 268.3321 121.92 0)
+			(at 40.3972 21.59 0)
 			(effects
 				(font
@@
 		)
 	)
-	(global_label "Vcc_IO8"
+	(global_label "VCORE_3V3"
 		(shape passive)
-		(at 198.12 121.92 0)
+		(at 252.73 85.09 0)
 		(fields_autoplaced yes)
 		(effects
@@
 		)
 		(property "Intersheetrefs" "${INTERSHEET_REFS}"
-			(at 207.3721 121.92 0)
+			(at 265.1872 85.09 0)
 			(effects
 				(font
@@
 		)
 	)
-	(global_label "Vcc_IO8"
-		(shape passive)
-		(at 255.27 58.42 0)
+	(global_label "FPGA_USB_RTSn"
+		(shape input)
+		(at 62.23 29.21 0)
 		(fields_autoplaced yes)
 		(effects
@@
 		)
 		(property "Intersheetrefs" "${INTERSHEET_REFS}"
-			(at 264.5221 58.42 0)
+			(at 80.2737 29.21 0)
 			(effects
 				(font
@@
 		)
 	)
-	(global_label "Vcc_IO8"
+	(global_label "VCORE_3V3"
 		(shape passive)
-		(at 219.71 26.67 180)
-		(fields_autoplaced yes)
-		(effects
-			(font
-				(size 1.27 1.27)
-			)
-			(justify right)
-		)
-		(property "Intersheetrefs" "${INTERSHEET_REFS}"
-			(at 210.4579 26.67 0)
-			(effects
-				(font
-					(size 1.27 1.27)
-				)
-				(justify right)
-				(hide yes)
-			)
-		)
-	)
-	(global_label "Vcc_IO8"
-		(shape passive)
-		(at 255.27 85.09 0)
+		(at 198.12 120.65 0)
 		(fields_autoplaced yes)
 		(effects
@@
 		)
 		(property "Intersheetrefs" "${INTERSHEET_REFS}"
-			(at 264.5221 85.09 0)
+			(at 210.5772 120.65 0)
 			(effects
 				(font
@@
 		)
 	)
-	(global_label "Vcc_IO8"
+	(global_label "VCORE_3V3"
 		(shape passive)
-		(at 241.3 119.38 0)
+		(at 252.73 58.42 0)
 		(fields_autoplaced yes)
 		(effects
@@
 		)
 		(property "Intersheetrefs" "${INTERSHEET_REFS}"
-			(at 250.5521 119.38 0)
+			(at 265.1872 58.42 0)
 			(effects
 				(font
@@
 		)
 	)
-	(global_label "Vcc_IO8"
+	(global_label "VCORE_3V3"
 		(shape passive)
-		(at 31.75 21.59 0)
+		(at 259.08 121.92 0)
 		(fields_autoplaced yes)
 		(effects
@@
 		)
 		(property "Intersheetrefs" "${INTERSHEET_REFS}"
-			(at 41.0021 21.59 0)
+			(at 271.5372 121.92 0)
 			(effects
 				(font
@@
 		(dnp no)
 		(property "Reference" "IC1"
-			(at 38.1 20.32 0)
+			(at 42.926 21.082 0)
 			(effects
 				(font
@@
 		)
 		(property "Value" "ECP5-BGA256"
-			(at 38.1 22.86 0)
+			(at 40.386 24.13 0)
 			(effects
 				(font
@@
 			)
 		)
-		(property "Footprint" "BGA256C80P16X16_1400X1400X170"
+		(property "Footprint" "fpga:BGA256C80P16X16_1400X1400X170"
 			(at -44.45 -21.59 0)
 			(effects
@@
 			)
 		)
-		(property "Description" "FPGA - Field Programmable Gate Array ECP5; 12k LUTs; 1.1V"
+		(property "Description" "FPGA - Field Programmable Gate Array ECP5; 25k LUTs; 1.1V"
 			(at -55.88 -43.18 0)
 			(effects
@@
 			)
 		)
-		(property "Part Number" "LFE5U-12F-6BG256C"
+		(property "Part Number" "LFE5U-25F-6BG256C "
+			(at -54.61 -64.77 0)
+			(effects
+				(font
+					(size 1.27 1.27)
+				)
+				(justify left)
+				(hide yes)
+			)
+		)
+		(property "LPN" "C1521614"
 			(at -54.61 -64.77 0)
 			(effects
@@
 			)
 		)
+		(property "MPN" "LFE5U-25F-6BG256C "
+			(at 36.83 66.04 0)
+			(effects
+				(font
+					(size 1.27 1.27)
+				)
+				(hide yes)
+			)
+		)
 		(pin "N4"
 		)
@@
 			(effects
 				(font
-					(size 1.27 1.27)
-				)
-				(hide yes)
-			)
-		)
-		(property "LCSC Part Number" ""
-			(at 190.5 139.7 0)
-			(effects
-				(font
-					(size 1.27 1.27)
-				)
-				(hide yes)
-			)
-		)
-		(property "Manufacturing Part Number" ""
-			(at 190.5 139.7 0)
-			(effects
-				(font
