File: acoustic-carrier-hw/acoustic-carrier-board/acoustic-carrier-board.kicad_pcb (KiCad board)
At the start: 6 copper layers, 374 parts, among them IC1 ECP5-BGA256, IC1101 MT41K256M16TW-107_P, J1001 BWU.FL-IPEX1, J1002 BWU.FL-IPEX1, J1003 BWU.FL-IPEX1, J1004 BWU.FL-IPEX1, J1005 BWU.FL-IPEX1, J1006 BWU.FL-IPEX1, J1007 8P8C_Shielded, J1008 BWU.FL-IPEX1, J1201 HR911130A, J201 Conn_02x08_Odd_Even, J701 Conn_01x10_Socket, J702 Conn_01x08_Socket, J801 TYPE-C-31-M-12, J901 Conn_02x08_Odd_Even, Q201 AO3401A, U1001 MS9280, U1002 THS4521IDGK, U1003 DGQ2788AEN-T1-GE4, U1004 LMV321, U1005 TL432DBZ, U1201 KSZ9031RN, U201 TPS2121RUX, U202 TLV62569DBV, U203 TLV62569DBV, U204 TLV62569DBV, U205 TLV62569DBV, U206 OPA376xxDBV, U701 W25Q128JVS, U702 W25Q128JVS, U801 USB3300-EZK, U802 TS3USB30EDGSR, U805 LMV321, Y1201 25MHz, Y601 Crystal Oscillator, Y801 Crystal_GND24_Small

Commit message: [¢arrier] Added netties and determined trace geometry for 50 ohms SE / 100 ohms DIFF impedance (next) reset the appropriate DQS group signals, RGMII and USB signals
Parts:
- added NT401: NetTie_2, iw-misc:NetTie-2_SMD_Pad0.1565mm, F.Cu at (158.1, 108.9)
- added NT402: NetTie_2, iw-misc:NetTie-2_SMD_Pad0.1565mm, F.Cu at (158.1, 110.4)
- added NT403: NetTie_2, iw-misc:NetTie-2_SMD_Pad0.1565mm, F.Cu at (158.1, 111.9)
- added NT404: NetTie_2, iw-misc:NetTie-2_SMD_Pad0.1565mm, F.Cu at (158.1, 113.4)
- added NT405: NetTie_2, iw-misc:NetTie-2_SMD_Pad0.1565mm, F.Cu at (158.1, 114.9)
- added NT406: NetTie_2, iw-misc:NetTie-2_SMD_Pad0.1565mm, F.Cu at (159.8, 108.9)
- added NT407: NetTie_2, iw-misc:NetTie-2_SMD_Pad0.1565mm, F.Cu at (159.8, 110.4)
- added NT408: NetTie_2, iw-misc:NetTie-2_SMD_Pad0.1565mm, F.Cu at (159.8, 111.9)
- added NT409: NetTie_2, iw-misc:NetTie-2_SMD_Pad0.1565mm, F.Cu at (159.8, 113.4)
- added NT410: NetTie_2, iw-misc:NetTie-2_SMD_Pad0.1565mm, F.Cu at (159.8, 114.9)
- added NT415: NetTie_2, iw-misc:NetTie-2_SMD_Pad0.1565mm, F.Cu at (161.6, 108.9)
- added NT416: NetTie_2, iw-misc:NetTie-2_SMD_Pad0.1565mm, F.Cu at (161.6, 110.4)
- added NT417: NetTie_2, iw-misc:NetTie-2_SMD_Pad0.1565mm, F.Cu at (161.6, 111.9)
- added NT418: NetTie_2, iw-misc:NetTie-2_SMD_Pad0.1565mm, F.Cu at (161.6, 113.4)
- added NT502: NetTie_2, iw-misc:NetTie-2_SMD_Pad0.1565mm, F.Cu at (158.1, 97.9)
- added NT503: NetTie_2, iw-misc:NetTie-2_SMD_Pad0.1565mm, F.Cu at (158.1, 99.4)
- added NT504: NetTie_2, iw-misc:NetTie-2_SMD_Pad0.1565mm, F.Cu at (158.1, 100.9)
- added NT505: NetTie_2, iw-misc:NetTie-2_SMD_Pad0.1240mm, F.Cu at (163.3, 97.9)
- added NT506: NetTie_2, iw-misc:NetTie-2_SMD_Pad0.1240mm, F.Cu at (163.3, 99.4)
- added NT507: NetTie_2, iw-misc:NetTie-2_SMD_Pad0.1565mm, F.Cu at (158.1, 102.4)
- added NT508: NetTie_2, iw-misc:NetTie-2_SMD_Pad0.1565mm, F.Cu at (158.1, 103.9)
- added NT509: NetTie_2, iw-misc:NetTie-2_SMD_Pad0.1565mm, F.Cu at (158.1, 105.4)
- added NT510: NetTie_2, iw-misc:NetTie-2_SMD_Pad0.1565mm, F.Cu at (159.8, 97.9)
- added NT511: NetTie_2, iw-misc:NetTie-2_SMD_Pad0.1565mm, F.Cu at (159.8, 99.4)
- added NT513: NetTie_2, iw-misc:NetTie-2_SMD_Pad0.1565mm, F.Cu at (159.8, 100.9)
- added NT514: NetTie_2, iw-misc:NetTie-2_SMD_Pad0.1565mm, F.Cu at (159.8, 102.4)
- added NT515: NetTie_2, iw-misc:NetTie-2_SMD_Pad0.1565mm, F.Cu at (159.8, 103.9)
- added NT516: NetTie_2, iw-misc:NetTie-2_SMD_Pad0.1565mm, F.Cu at (159.8, 105.4)
- added NT517: NetTie_2, iw-misc:NetTie-2_SMD_Pad0.1565mm, F.Cu at (161.6, 97.9)
- added NT518: NetTie_2, iw-misc:NetTie-2_SMD_Pad0.1565mm, F.Cu at (161.6, 99.4)
- added NT519: NetTie_2, iw-misc:NetTie-2_SMD_Pad0.1565mm, F.Cu at (161.6, 100.9)
- added NT520: NetTie_2, iw-misc:NetTie-2_SMD_Pad0.1565mm, F.Cu at (161.6, 102.4)
- added NT521: NetTie_2, iw-misc:NetTie-2_SMD_Pad0.1240mm, F.Cu at (163.3, 100.9)
- added NT522: NetTie_2, iw-misc:NetTie-2_SMD_Pad0.1240mm, F.Cu at (163.3, 102.4)
- added NT523: NetTie_2, iw-misc:NetTie-2_SMD_Pad0.1565mm, F.Cu at (161.6, 103.9)
- added NT524: NetTie_2, iw-misc:NetTie-2_SMD_Pad0.1565mm, F.Cu at (161.6, 105.4)
- added NT601: NetTie_2, iw-misc:NetTie-2_SMD_Pad0.1565mm, F.Cu at (147.2, 97.9)
- added NT602: NetTie_2, iw-misc:NetTie-2_SMD_Pad0.1565mm, F.Cu at (147.2, 99.4)
- added NT603: NetTie_2, iw-misc:NetTie-2_SMD_Pad0.1565mm, F.Cu at (147.2, 100.9)
- added NT604: NetTie_2, iw-misc:NetTie-2_SMD_Pad0.1565mm, F.Cu at (147.2, 102.4)
- added NT605: NetTie_2, iw-misc:NetTie-2_SMD_Pad0.1565mm, F.Cu at (147.2, 103.9)
- added NT606: NetTie_2, iw-misc:NetTie-2_SMD_Pad0.1565mm, F.Cu at (148.9, 97.9)
- added NT607: NetTie_2, iw-misc:NetTie-2_SMD_Pad0.1565mm, F.Cu at (148.9, 99.4)
- added NT608: NetTie_2, iw-misc:NetTie-2_SMD_Pad0.1565mm, F.Cu at (148.9, 100.9)
- added NT609: NetTie_2, iw-misc:NetTie-2_SMD_Pad0.1565mm, F.Cu at (148.9, 102.4)
- added NT610: NetTie_2, iw-misc:NetTie-2_SMD_Pad0.1565mm, F.Cu at (148.9, 103.9)
- added NT611: NetTie_2, iw-misc:NetTie-2_SMD_Pad0.1240mm, F.Cu at (147.1, 105.4)
- added NT612: NetTie_2, iw-misc:NetTie-2_SMD_Pad0.1240mm, F.Cu at (147.1, 106.9)
- added NT613: NetTie_2, iw-misc:NetTie-2_SMD_Pad0.1565mm, F.Cu at (150.7, 97.9)
- added NT614: NetTie_2, iw-misc:NetTie-2_SMD_Pad0.1565mm, F.Cu at (150.7, 99.4)
- added NT615: NetTie_2, iw-misc:NetTie-2_SMD_Pad0.1565mm, F.Cu at (150.7, 100.9)
- added NT616: NetTie_2, iw-misc:NetTie-2_SMD_Pad0.1565mm, F.Cu at (150.7, 102.4)
- added NT617: NetTie_2, iw-misc:NetTie-2_SMD_Pad0.1565mm, F.Cu at (150.7, 103.9)
- added NT618: NetTie_2, iw-misc:NetTie-2_SMD_Pad0.1565mm, F.Cu at (152.5, 97.9)
- added NT619: NetTie_2, iw-misc:NetTie-2_SMD_Pad0.1565mm, F.Cu at (152.5, 99.4)
- added NT620: NetTie_2, iw-misc:NetTie-2_SMD_Pad0.1565mm, F.Cu at (152.5, 100.9)
- added NT621: NetTie_2, iw-misc:NetTie-2_SMD_Pad0.1565mm, F.Cu at (152.5, 102.4)
- added NT622: NetTie_2, iw-misc:NetTie-2_SMD_Pad0.1565mm, F.Cu at (152.5, 103.9)
- added NT623: NetTie_2, iw-misc:NetTie-2_SMD_Pad0.1565mm, F.Cu at (154.3, 97.9)
- added NT624: NetTie_2, iw-misc:NetTie-2_SMD_Pad0.1565mm, F.Cu at (154.3, 99.4)
- added NT625: NetTie_2, iw-misc:NetTie-2_SMD_Pad0.1565mm, F.Cu at (154.3, 100.9)
- added NT626: NetTie_2, iw-misc:NetTie-2_SMD_Pad0.1565mm, F.Cu at (154.3, 102.4)
- added NT627: NetTie_2, iw-misc:NetTie-2_SMD_Pad0.1565mm, F.Cu at (154.3, 103.9)
- added R203: 24k, Resistor_SMD:R_0603_1608Metric, F.Cu at (265.7, 133.0)
Connections:
- IC1 pad A11: /ETHERNET-PHY/RGMII.CTL -> /FPGA-BANK-01/RX_RGMII_CTL
- IC1 pad A12: /ETHERNET-PHY/RGMII.D0 -> /FPGA-BANK-01/RX_RGMII_D0
- IC1 pad A13: /ETHERNET-PHY/RGMII.D3 -> /FPGA-BANK-01/TX_RGMII_D3
- IC1 pad A14: /ETHERNET-PHY/RGMII.CLK -> /FPGA-BANK-01/TX_RGMII_CLK
- IC1 pad A15: /ETHERNET-PHY/RGMII.CLK -> /FPGA-BANK-01/MDIO_RGMII_CLK
- IC1 pad B12: /ETHERNET-PHY/RGMII.D1 -> /FPGA-BANK-01/RX_RGMII_D1
- IC1 pad B13: /ETHERNET-PHY/RGMII.CTL -> /FPGA-BANK-01/TX_RGMII_CTL
- IC1 pad B14: /ETHERNET-PHY/RGMII.DATA -> /FPGA-BANK-01/MDIO_RGMII_DATA
- IC1 pad B15: /DDR3/DDR3.DQ1 -> /FPGA-DQBANK-23/DDR3_DQ1
- IC1 pad B16: /DDR3/DDR3.DQ0 -> /FPGA-DQBANK-23/DDR3_DQ0
- IC1 pad C12: /ETHERNET-PHY/RGMII.D2 -> /FPGA-BANK-01/RX_RGMII_D2
- IC1 pad C13: /ETHERNET-PHY/RGMII.D0 -> /FPGA-BANK-01/TX_RGMII_D0
- IC1 pad C14: /DDR3/DDR3.DQ2 -> /FPGA-DQBANK-23/DDR3_DQ2
- IC1 pad C15: /DDR3/DDR3.DQ5 -> /FPGA-DQBANK-23/DDR3_DQ5
- IC1 pad C16: /DDR3/DDR3.DQ4 -> /FPGA-DQBANK-23/DDR3_DQ4
- IC1 pad D12: /ETHERNET-PHY/RGMII.D3 -> /FPGA-BANK-01/RX_RGMII_D3
- IC1 pad D13: /ETHERNET-PHY/RGMII.D1 -> /FPGA-BANK-01/TX_RGMII_D1
- IC1 pad D14: /DDR3/DDR3.DQ3 -> /FPGA-DQBANK-23/DDR3_DQ3
- IC1 pad D16: /DDR3/DDR3.LDQS -> /FPGA-DQBANK-23/DDR3_LDQS
- IC1 pad E12: /ETHERNET-PHY/RGMII.CLK -> /FPGA-BANK-01/RX_RGMII_CLK
- IC1 pad E13: /ETHERNET-PHY/RGMII.D2 -> /FPGA-BANK-01/TX_RGMII_D2
- IC1 pad E14: /DDR3/DDR3.DQ6 -> /FPGA-DQBANK-23/DDR3_DQ6
- IC1 pad E15: /DDR3/DDR3.LDQS# -> /FPGA-DQBANK-23/DDR3_LDQS#
- IC1 pad F13: /DDR3/DDR3.LDM -> /FPGA-DQBANK-23/DDR3_LDM
- IC1 pad F14: /DDR3/DDR3.DQ7 -> /FPGA-DQBANK-23/DDR3_DQ7
- IC1 pad G16: /DDR3/DDR3.UDQS -> /FPGA-DQBANK-23/DDR3_UDQS
- IC1 pad H13: /DDR3/DDR3.DQ8 -> /FPGA-DQBANK-23/DDR3_DQ8
- IC1 pad H15: /DDR3/DDR3.UDQS# -> /FPGA-DQBANK-23/DDR3_UDQS#
- IC1 pad J12: /DDR3/DDR3.DQ10 -> /FPGA-DQBANK-23/DDR3_DQ10
- IC1 pad J13: /DDR3/DDR3.DQ9 -> /FPGA-DQBANK-23/DDR3_DQ9
- IC1 pad J14: /DDR3/DDR3.DQ11 -> /FPGA-DQBANK-23/DDR3_DQ11
- IC1 pad J15: /DDR3/DDR3.DQ14 -> /FPGA-DQBANK-23/DDR3_DQ14
- IC1 pad J16: /DDR3/DDR3.DQ13 -> /FPGA-DQBANK-23/DDR3_DQ13
- IC1 pad K14: /DDR3/DDR3.DQ12 -> /FPGA-DQBANK-23/DDR3_DQ12
- IC1 pad K15: /DDR3/DDR3.UDM -> /FPGA-DQBANK-23/DDR3_UDM
- IC1 pad K16: /DDR3/DDR3.DQ15 -> /FPGA-DQBANK-23/DDR3_DQ15
- IC1 pad K4: /DDR3/DDR3.A10 -> /FPGA-DQBANK-67/DDR3_A10
- IC1 pad K5: /DDR3/DDR3.A9 -> /FPGA-DQBANK-67/DDR3_A9
- IC1 pad L1: /DDR3/DDR3.A14 -> /FPGA-DQBANK-67/DDR3_A14
- IC1 pad L2: /DDR3/DDR3.A13 -> /FPGA-DQBANK-67/DDR3_A13
- IC1 pad L3: /DDR3/DDR3.A4 -> /FPGA-DQBANK-67/DDR3_A4
- IC1 pad L4: /DDR3/DDR3.A8 -> /FPGA-DQBANK-67/DDR3_A8
- IC1 pad L5: /DDR3/DDR3.A7 -> /FPGA-DQBANK-67/DDR3_A7
- IC1 pad M1: /DDR3/DDR3.A12 -> /FPGA-DQBANK-67/DDR3_A12
- IC1 pad M2: /DDR3/DDR3.A11 -> /FPGA-DQBANK-67/DDR3_A11
- IC1 pad M3: /DDR3/DDR3.A3 -> /FPGA-DQBANK-67/DDR3_A3
- IC1 pad M5: /DDR3/DDR3.WE# -> /FPGA-DQBANK-67/DDR3_WE#
- IC1 pad M6: /DDR3/DDR3.RAS# -> /FPGA-DQBANK-67/DDR3_RAS#
- IC1 pad N1: /DDR3/DDR3.A6 -> /FPGA-DQBANK-67/DDR3_A6
- IC1 pad N3: /DDR3/DDR3.A1 -> /FPGA-DQBANK-67/DDR3_A1
- IC1 pad N4: /DDR3/DDR3.A0 -> /FPGA-DQBANK-67/DDR3_A0
- IC1 pad N5: /DDR3/DDR3.RESET# -> /FPGA-DQBANK-67/DDR3_RESET#
- IC1 pad N6: /DDR3/DDR3.CK -> /FPGA-DQBANK-67/DDR3_CK
- IC1 pad P1: /DDR3/DDR3.A2 -> /FPGA-DQBANK-67/DDR3_A2
- IC1 pad P2: /DDR3/DDR3.A5 -> /FPGA-DQBANK-67/DDR3_A5
- IC1 pad P4: /DDR3/DDR3.BA2 -> /FPGA-DQBANK-67/DDR3_BA2
- IC1 pad P5: /DDR3/DDR3.CK# -> /FPGA-DQBANK-67/DDR3_CK#
- IC1 pad P6: /DDR3/DDR3.CKE -> /FPGA-DQBANK-67/DDR3_CKE
- IC1 pad R3: /DDR3/DDR3.BA1 -> /FPGA-DQBANK-67/DDR3_BA1
- IC1 pad R4: /DDR3/DDR3.BA0 -> /FPGA-DQBANK-67/DDR3_BA0
- IC1 pad R5: /DDR3/DDR3.ODT -> /FPGA-DQBANK-67/DDR3_ODT
- IC1 pad T3: /DDR3/DDR3.CAS# -> /FPGA-DQBANK-67/DDR3_CAS#
- IC1 pad T4: /DDR3/DDR3.CS# -> /FPGA-DQBANK-67/DDR3_CS#

Commit message: [carrier] Removed USB-switch, placed decouplpling for DDR3 and ECP5U (next) consider adding buffers on CC1 and CC2 pins
Parts:
- removed C1116, C1117, C505, C506, C604, C605, C608, C801, C823, C824: 0.1uF, Capacitor_SMD:C_0402_1005Metric
- removed C504, C607: 4.7uF, Capacitor_SMD:C_0402_1005Metric
- removed C606, C802: 10nF, Capacitor_SMD:C_0402_1005Metric
- removed L601: 120@100MHz, Inductor_SMD:L_0603_1608Metric
- removed NT401, NT402, NT403, NT404, NT405, NT406, NT407, NT408, NT409, NT410, NT415, NT416, NT417, NT418, NT502, NT503, NT504, NT507, NT508, NT509, NT510, NT511, NT513, NT514, NT515, NT516, NT517, NT518, NT519, NT520, NT523, NT524, NT601, NT602, NT603, NT604, NT605, NT606, NT607, NT608, NT609, NT610, NT613, NT614, NT615, NT616, NT617, NT618, NT619, NT620, NT621, NT622, NT623, NT624, NT625, NT626, NT627: NetTie_2, iw-misc:NetTie-2_SMD_Pad0.1565mm
- removed NT505, NT506, NT521, NT522, NT611, NT612: NetTie_2, iw-misc:NetTie-2_SMD_Pad0.1240mm
- removed R802: 51, Resistor_SMD:R_0603_1608Metric
- removed R803, R825: 10k, Resistor_SMD:R_0603_1608Metric
- removed R819: 240k, Resistor_SMD:R_0603_1608Metric
- removed R822: 9k1, Resistor_SMD:R_0603_1608Metric_Pad0.98x0.95mm_HandSolder
- removed R823, R824, R828, R831: 1M, Resistor_SMD:R_0603_1608Metric_Pad0.98x0.95mm_HandSolder
- removed R827: 560, Resistor_SMD:R_0603_1608Metric_Pad0.98x0.95mm_HandSolder
- removed R829: 1k, Resistor_SMD:R_0603_1608Metric
- removed TP808, TP809, TP810: TestPoint, TestPoint:TestPoint_Loop_D1.80mm_Drill1.0mm_Beaded
- removed U802: TS3USB30EDGSR, Package_SO:VSSOP-10_3x3mm_P0.5mm
- removed U805: LMV321, Package_TO_SOT_SMD:SOT-23-5
- removed U806: ~, Package_TO_SOT_SMD:SOT-23-5
- added C1118: 0.1uF, Capacitor_SMD:C_0201_0603Metric, B.Cu at (125.9, 89.3)
- added C1119: 0.1uF, Capacitor_SMD:C_0201_0603Metric, B.Cu at (126.4, 84.9)
- added C1120: 0.1uF, Capacitor_SMD:C_0201_0603Metric, B.Cu at (120.4, 91.7)
- added C1121: 0.1uF, Capacitor_SMD:C_0201_0603Metric, B.Cu at (119.6, 87.7)
- added C1122: 0.1uF, Capacitor_SMD:C_0201_0603Metric, B.Cu at (124.4, 91.7)
- added C1123: 0.1uF, Capacitor_SMD:C_0201_0603Metric, B.Cu at (120.0, 82.5)
- added C1124: 0.1uF, Capacitor_SMD:C_0201_0603Metric, B.Cu at (126.9, 91.7)
- added C1125: 0.1uF, Capacitor_SMD:C_0201_0603Metric, B.Cu at (120.1, 84.1)
- added C509: 0.1uF, Capacitor_SMD:C_0201_0603Metric, B.Cu at (122.8, 71.1)
- added C510: 0.1uF, Capacitor_SMD:C_0201_0603Metric, B.Cu at (123.2, 72.2)
- added C511: 10nF, Capacitor_SMD:C_0201_0603Metric, B.Cu at (122.0, 71.8)
- added C512: 4.7uF, Capacitor_SMD:C_0402_1005Metric, B.Cu at (116.8, 68.1)
- added C513: 0.1uF, Capacitor_SMD:C_0201_0603Metric, B.Cu at (118.5, 75.5)
- added C611: 4.7uF, Capacitor_SMD:C_0402_1005Metric, B.Cu at (165.4, 106.3)
- added C612: 0.1uF, Capacitor_SMD:C_0201_0603Metric, B.Cu at (165.4, 104.3)
- added C613: 0.1uF, Capacitor_SMD:C_0201_0603Metric, B.Cu at (165.4, 102.3)
- added L502: 120@100MHz, Inductor_SMD:L_0603_1608Metric, B.Cu at (114.5, 68.7)
- C1002, C1003, C1004, C1005, C1008, C1010, C1011, C1013, C1019, C1021, C1203, C1204, C1206, C1207, C1209, C1210, C1211, C1212, C1213, C1214, C1216, C1217, C1218, C1219, C1220, C1221, C1222, C1223, C1225, C1229, C301, C302, C303, C304, C305, C306, C310, C311, C404, C405, C609, C704, C706: footprint Capacitor_SMD:C_0402_1005Metric -> Capacitor_SMD:C_0201_0603Metric
- C1101, C1102, C1103, C1104, C1105, C1106, C1108, C1109, C1110, C1111, C1112, C1114, C1115, C401, C402, C501, C502, C507, C508, C601, C602, C702, C703, C807, C808, C809, C810, C811, C812, C816, C817, C820, C821, C822, C825: footprint Capacitor_SMD:C_0402_1005Metric -> Capacitor_SMD:C_0201_0603Metric; moved to B.Cu
- C1107, C1113, C403, C503, C603, C701, C804, C805, C813, C814, C819, D801, D802, L1101, L1102, L501, R1101, R801, R804, R805, R808, R809, R810, R811, R812, R813, R814, R815, R816, R817, R818, R820, R821, R826, R830, TP804, TP805, TP806, TP807, U803, U804: moved to B.Cu
- C1226: value 0.1uF -> 100 nF +-5%
- moved C503 288.8 mm to (116.8, 70.0), turned to 90 degrees
- moved C502 285.7 mm to (124.4, 71.1), turned to 90 degrees
- moved C501 283.7 mm to (123.6, 71.1), turned to 90 degrees
- moved L501 282.3 mm to (114.5, 70.4), turned to 180 degrees
- moved C508 258.8 mm to (125.3, 73.5), turned to 90 degrees
- moved C507 256.8 mm to (124.6, 73.5), turned to 90 degrees
- moved R1003 248.9 mm to (259.1, 65.7)
- moved R1002 244.8 mm to (255.8, 65.7)
- moved R1005 242.4 mm to (258.6, 84.4), turned to 180 degrees
- moved C603 240.5 mm to (134.6, 72.3)
- moved C703 238.8 mm to (122.4, 67.4)
- moved R1004 238.3 mm to (255.3, 84.5)
- moved C702 237.5 mm to (122.3, 66.7)
- moved C602 237.2 mm to (134.4, 73.6)
- moved R1008 237.0 mm to (228.9, 24.6)
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Connections:
- net /FPGA-DQBANK-23/VDDR_BANK renamed /FPGA-DQBANK-23/VDDR_BANK2
- C1102 pad 1: /DDR3/VDDR_CORE -> /DDR3/VDDR_DQ
- IC1 pad A11: /FPGA-BANK-01/RX_RGMII_CTL -> /ETHERNET-PHY/RGMII_RX.CTL
- IC1 pad A12: /FPGA-BANK-01/RX_RGMII_D0 -> /ETHERNET-PHY/RGMII_RX.D0
- IC1 pad A13: /FPGA-BANK-01/TX_RGMII_D3 -> /ETHERNET-PHY/RGMII_TX.D3
- IC1 pad A14: /FPGA-BANK-01/TX_RGMII_CLK -> /ETHERNET-PHY/RGMII_TX.CLK
- IC1 pad A15: /FPGA-BANK-01/MDIO_RGMII_CLK -> /ETHERNET-PHY/RGMII_MDIO.CLK
- IC1 pad B12: /FPGA-BANK-01/RX_RGMII_D1 -> /ETHERNET-PHY/RGMII_RX.D1
- IC1 pad B13: /FPGA-BANK-01/TX_RGMII_CTL -> /ETHERNET-PHY/RGMII_TX.CTL
- IC1 pad B14: /FPGA-BANK-01/MDIO_RGMII_DATA -> /ETHERNET-PHY/RGMII_MDIO.DATA
- IC1 pad B15: /FPGA-DQBANK-23/DDR3_DQ1 -> /DDR3/DDR3.DQ1
- IC1 pad B16: /FPGA-DQBANK-23/DDR3_DQ0 -> /DDR3/DDR3.DQ0
- IC1 pad C12: /FPGA-BANK-01/RX_RGMII_D2 -> /ETHERNET-PHY/RGMII_RX.D2
- IC1 pad C13: /FPGA-BANK-01/TX_RGMII_D0 -> /ETHERNET-PHY/RGMII_TX.D0
- IC1 pad C14: /FPGA-DQBANK-23/DDR3_DQ2 -> /DDR3/DDR3.DQ2
- IC1 pad C15: /FPGA-DQBANK-23/DDR3_DQ5 -> /DDR3/DDR3.DQ5
- IC1 pad C16: /FPGA-DQBANK-23/DDR3_DQ4 -> /DDR3/DDR3.DQ4
- IC1 pad D12: /FPGA-BANK-01/RX_RGMII_D3 -> /ETHERNET-PHY/RGMII_RX.D3
- IC1 pad D13: /FPGA-BANK-01/TX_RGMII_D1 -> /ETHERNET-PHY/RGMII_TX.D1
- IC1 pad D14: /FPGA-DQBANK-23/DDR3_DQ3 -> /DDR3/DDR3.DQ3
- IC1 pad D16: /FPGA-DQBANK-23/DDR3_LDQS -> /DDR3/DDR3.LDQS
- IC1 pad E12: /FPGA-BANK-01/RX_RGMII_CLK -> /ETHERNET-PHY/RGMII_RX.CLK
- IC1 pad E13: /FPGA-BANK-01/TX_RGMII_D2 -> /ETHERNET-PHY/RGMII_TX.D2
- IC1 pad E14: /FPGA-DQBANK-23/DDR3_DQ6 -> /DDR3/DDR3.DQ6
- IC1 pad E15: /FPGA-DQBANK-23/DDR3_LDQS# -> /DDR3/DDR3.LDQS#
- IC1 pad E16: unconnected-(IC1D-PR11D/RDQ8-PadE16) -> /DDR3/DDR3.LDM
- IC1 pad F13: /FPGA-DQBANK-23/DDR3_LDM -> unconnected-(IC1D-PR8C-PadF13)
- IC1 pad F14: /FPGA-DQBANK-23/DDR3_DQ7 -> unconnected-(IC1D-PR5D-PadF14)
- IC1 pad F15: unconnected-(IC1D-PR11C-PadF15) -> /DDR3/DDR3.DQ7
- IC1 pad F16: unconnected-(IC1D-PR14A/RDQ20-PadF16) -> /DDR3/DDR3.DQ8
- IC1 pad G15: unconnected-(IC1D-PR14B-PadG15) -> /DDR3/DDR3.DQ9
- IC1 pad G16: /FPGA-DQBANK-23/DDR3_UDQS -> /DDR3/DDR3.UDQS
- IC1 pad H13: /FPGA-DQBANK-23/DDR3_DQ8 -> unconnected-(IC1D-PR17B-PadH13)
- IC1 pad H14: unconnected-(IC1D-PR14D-PadH14) -> /DDR3/DDR3.DQ10
- IC1 pad H15: /FPGA-DQBANK-23/DDR3_UDQS# -> /DDR3/DDR3.UDQS#
- IC1 pad J12: /FPGA-DQBANK-23/DDR3_DQ10 -> unconnected-(IC1D-PR17D-PadJ12)
- IC1 pad J13: /FPGA-DQBANK-23/DDR3_DQ9 -> unconnected-(IC1D-PR17C-PadJ13)
- IC1 pad J14: /FPGA-DQBANK-23/DDR3_DQ11 -> /DDR3/DDR3.DQ11
- IC1 pad J15: /FPGA-DQBANK-23/DDR3_DQ14 -> /DDR3/DDR3.DQ14
- IC1 pad J16: /FPGA-DQBANK-23/DDR3_DQ13 -> /DDR3/DDR3.DQ13
- IC1 pad J6: /FPGA-DQBANK-67/VDDR_BANK -> VCORE_3V3
- IC1 pad J7: /FPGA-DQBANK-67/VDDR_BANK -> VCORE_3V3
- IC1 pad K11: VCORE_3V3 -> /FPGA-DQBANK-23/VDDR_BANK3
- IC1 pad K13: /FPGA-DQBANK-23/USB.CLK -> /DDR3/DDR3.A10
- IC1 pad K14: /FPGA-DQBANK-23/DDR3_DQ12 -> /DDR3/DDR3.DQ12
- IC1 pad K15: /FPGA-DQBANK-23/DDR3_UDM -> /DDR3/DDR3.UDM
- IC1 pad K16: /FPGA-DQBANK-23/DDR3_DQ15 -> /DDR3/DDR3.DQ15
- IC1 pad K4: /FPGA-DQBANK-67/DDR3_A10 -> /FPGA-DQBANK-67/USB.CLK
- IC1 pad K5: /FPGA-DQBANK-67/DDR3_A9 -> unconnected-(IC1F-PL29B-PadK5)
- IC1 pad L1: /FPGA-DQBANK-67/DDR3_A14 -> unconnected-(IC1F-PL26A/LDQ32/PCLKT6_1-PadL1)
- IC1 pad L11: VCORE_3V3 -> /FPGA-DQBANK-23/VDDR_BANK3
- IC1 pad L14: /FPGA-DQBANK-23/USB.STP -> /DDR3/DDR3.A7
- IC1 pad L15: unconnected-(IC1E-PR26B/PCLKC3_1-PadL15) -> /DDR3/DDR3.A13
- IC1 pad L16: unconnected-(IC1E-PR26A/PCLKT3_1/RDQ32-PadL16) -> /DDR3/DDR3.A14
- IC1 pad L2: /FPGA-DQBANK-67/DDR3_A13 -> unconnected-(IC1F-PL26B/PCLKC6_1-PadL2)
- IC1 pad L3: /FPGA-DQBANK-67/DDR3_A4 -> /FPGA-DQBANK-67/USB.STP
- IC1 pad L4: /FPGA-DQBANK-67/DDR3_A8 -> unconnected-(IC1F-PL29C/PL29C-PadL4)
- IC1 pad L5: /FPGA-DQBANK-67/DDR3_A7 -> unconnected-(IC1F-PL29D-PadL5)
- IC1 pad M1: /FPGA-DQBANK-67/DDR3_A12 -> unconnected-(IC1F-PL26C/PCLKT6_0-PadM1)
- IC1 pad M11: unconnected-(IC1E-PR47A-PadM11) -> /DDR3/DDR3.RAS#
- IC1 pad M12: unconnected-(IC1E-PR44C-PadM12) -> /DDR3/DDR3.BA0
- IC1 pad M13: /FPGA-DQBANK-23/USB.D1 -> unconnected-(IC1E-PR35C-PadM13)
- IC1 pad M14: /FPGA-DQBANK-23/USB.DIR -> /DDR3/DDR3.A6
- IC1 pad M15: unconnected-(IC1E-PR26D/PCLKC3_0-PadM15) -> /DDR3/DDR3.A11
- IC1 pad M16: unconnected-(IC1E-PR26C/PCLKT3_0-PadM16) -> /DDR3/DDR3.A12
- IC1 pad M2: /FPGA-DQBANK-67/DDR3_A11 -> unconnected-(IC1F-PL26D/PCLKC6_0-PadM2)
- IC1 pad M3: /FPGA-DQBANK-67/DDR3_A3 -> /FPGA-DQBANK-67/USB.DIR
- IC1 pad M4: unconnected-(IC1F-PL35C-PadM4) -> /FPGA-DQBANK-67/USB.D1
- IC1 pad M5: /FPGA-DQBANK-67/DDR3_WE# -> FPGA_CC1
- IC1 pad M6: /FPGA-DQBANK-67/DDR3_RAS# -> unconnected-(IC1F-PL47A-PadM6)
- IC1 pad N1: /FPGA-DQBANK-67/DDR3_A6 -> /FPGA-DQBANK-67/USB.RST
- IC1 pad N11: unconnected-(IC1E-PR47B-PadN11) -> /DDR3/DDR3.CK
- IC1 pad N12: unconnected-(IC1E-PR44D-PadN12) -> /DDR3/DDR3.CAS#
- IC1 pad N13: /FPGA-DQBANK-23/USB.D3 -> /DDR3/DDR3.A3
- IC1 pad N14: /FPGA-DQBANK-23/USB.D2 -> /DDR3/DDR3.A4
- IC1 pad N16: /FPGA-DQBANK-23/USB.RST -> /DDR3/DDR3.A9
- IC1 pad N3: /FPGA-DQBANK-67/DDR3_A1 -> /FPGA-DQBANK-67/USB.D2
- IC1 pad N4: /FPGA-DQBANK-67/DDR3_A0 -> /FPGA-DQBANK-67/USB.D3
- IC1 pad N5: /FPGA-DQBANK-67/DDR3_RESET# -> FPGA_CC2
- IC1 pad N6: /FPGA-DQBANK-67/DDR3_CK -> unconnected-(IC1F-PL47B-PadN6)
- IC1 pad P1: /FPGA-DQBANK-67/DDR3_A2 -> /FPGA-DQBANK-67/USB.NXT
- IC1 pad P11: unconnected-(IC1E-PR47C/LRC_GPLL0T_IN-PadP11) -> /DDR3/DDR3.CK#
- IC1 pad P12: unconnected-(IC1E-PR47D/LRC_GPLL0C_IN/RDQ44-PadP12) -> /DDR3/DDR3.CKE
- IC1 pad P13: /FPGA-DQBANK-23/USB.D7 -> /DDR3/DDR3.ODT
- IC1 pad P14: /FPGA-DQBANK-23/USB.D4 -> /DDR3/DDR3.A2
- IC1 pad P15: unconnected-(IC1E-PR32B/RDQSN32-PadP15) -> /DDR3/DDR3.A8
- IC1 pad P16: /FPGA-DQBANK-23/USB.NXT -> /DDR3/DDR3.A5
- IC1 pad P2: /FPGA-DQBANK-67/DDR3_A5 -> unconnected-(IC1F-PL32B/LDQSN32-PadP2)
- IC1 pad P3: unconnected-(IC1F-PL38B-PadP3) -> /FPGA-DQBANK-67/USB.D4
- IC1 pad P4: /FPGA-DQBANK-67/DDR3_BA2 -> FPGA_USB_SENSE
- IC1 pad P5: /FPGA-DQBANK-67/DDR3_CK# -> unconnected-(IC1F-PL47D/LLC_GPLL0C_IN-PadP5)
- IC1 pad P6: /FPGA-DQBANK-67/DDR3_CKE -> unconnected-(IC1F-PL47C/LLC_GPLL0T_IN-PadP6)
- IC1 pad R1: VDRR3L_V675 -> /FPGA-DQBANK-67/USB.D0
- IC1 pad R12: FPGA_USB_SENSE -> /DDR3/DDR3.BA2
- IC1 pad R13: FPGA_CC1 -> /DDR3/DDR3.WE#
- IC1 pad R14: unconnected-(IC1E-PR41B-PadR14) -> /DDR3/DDR3.CS#
- IC1 pad R15: /FPGA-DQBANK-23/USB.D5 -> /DDR3/DDR3.A1
- IC1 pad R16: /FPGA-DQBANK-23/USB.D0 -> VDRR3L_V675
- IC1 pad R2: unconnected-(IC1F-PL38C-PadR2) -> /FPGA-DQBANK-67/USB.D5
- IC1 pad R3: /FPGA-DQBANK-67/DDR3_BA1 -> unconnected-(IC1F-PL41B-PadR3)
- IC1 pad R4: /FPGA-DQBANK-67/DDR3_BA0 -> unconnected-(IC1F-PL41C-PadR4)
- IC1 pad R5: /FPGA-DQBANK-67/DDR3_ODT -> /FPGA-DQBANK-67/USB.D7
- IC1 pad T13: unconnected-(IC1E-PR44B/RDQSN44-PadT13) -> /DDR3/DDR3.BA1
- IC1 pad T14: FPGA_CC2 -> /DDR3/DDR3.RESET#
- IC1 pad T15: /FPGA-DQBANK-23/USB.D6 -> /DDR3/DDR3.A0
- IC1 pad T2: unconnected-(IC1F-PL38D-PadT2) -> /FPGA-DQBANK-67/USB.D6
- IC1 pad T3: /FPGA-DQBANK-67/DDR3_CAS# -> unconnected-(IC1F-PL41D-PadT3)
- IC1 pad T4: /FPGA-DQBANK-67/DDR3_CS# -> unconnected-(IC1F-PL44B/LDQSN44-PadT4)
- J801 pad A6: /USB-PHY/USB_DP1 -> /USB-PHY/USB_DP
- J801 pad A7: /USB-PHY/USB_DN1 -> /USB-PHY/USB_DM
- J801 pad B6: /USB-PHY/USB_DP2 -> /USB-PHY/USB_DP
- J801 pad B7: /USB-PHY/USB_DN2 -> /USB-PHY/USB_DM
- R1203 pad 2: /ETHERNET-PHY/RGMII.CLK -> /ETHERNET-PHY/RGMII_RX.CLK
- R1204 pad 1: /ETHERNET-PHY/RGMII.CTL -> /ETHERNET-PHY/RGMII_RX.CTL
- R1205 pad 1: /ETHERNET-PHY/RGMII.DATA -> /ETHERNET-PHY/RGMII_MDIO.DATA
- R1211 pad 1: /ETHERNET-PHY/RGMII.CLK -> /ETHERNET-PHY/RGMII_RX.CLK
- RN1201 pad 1: /ETHERNET-PHY/RGMII.D0 -> /ETHERNET-PHY/RGMII_RX.D0
- RN1201 pad 2: /ETHERNET-PHY/RGMII.D1 -> /ETHERNET-PHY/RGMII_RX.D1
- RN1201 pad 3: /ETHERNET-PHY/RGMII.D2 -> /ETHERNET-PHY/RGMII_RX.D2
- RN1201 pad 4: /ETHERNET-PHY/RGMII.D3 -> /ETHERNET-PHY/RGMII_RX.D3
- U1201 pad 19: /ETHERNET-PHY/RGMII.D0 -> /ETHERNET-PHY/RGMII_TX.D0
- U1201 pad 20: /ETHERNET-PHY/RGMII.D1 -> /ETHERNET-PHY/RGMII_TX.D1
- U1201 pad 21: /ETHERNET-PHY/RGMII.D2 -> /ETHERNET-PHY/RGMII_TX.D2
- U1201 pad 22: /ETHERNET-PHY/RGMII.D3 -> /ETHERNET-PHY/RGMII_TX.D3
- U1201 pad 24: /ETHERNET-PHY/RGMII.CLK -> /ETHERNET-PHY/RGMII_TX.CLK
- U1201 pad 25: /ETHERNET-PHY/RGMII.CTL -> /ETHERNET-PHY/RGMII_TX.CTL
- U1201 pad 27: /ETHERNET-PHY/RGMII.D3 -> /ETHERNET-PHY/RGMII_RX.D3
- U1201 pad 28: /ETHERNET-PHY/RGMII.D2 -> /ETHERNET-PHY/RGMII_RX.D2
- U1201 pad 31: /ETHERNET-PHY/RGMII.D1 -> /ETHERNET-PHY/RGMII_RX.D1
- U1201 pad 32: /ETHERNET-PHY/RGMII.D0 -> /ETHERNET-PHY/RGMII_RX.D0
- U1201 pad 33: /ETHERNET-PHY/RGMII.CTL -> /ETHERNET-PHY/RGMII_RX.CTL
- U1201 pad 35: /ETHERNET-PHY/RGMII.CLK -> /ETHERNET-PHY/RGMII_RX.CLK
- U1201 pad 36: /ETHERNET-PHY/RGMII.CLK -> /ETHERNET-PHY/RGMII_MDIO.CLK
- U1201 pad 37: /ETHERNET-PHY/RGMII.DATA -> /ETHERNET-PHY/RGMII_MDIO.DATA
- U801 pad 11: /FPGA-DQBANK-23/USB.NXT -> /FPGA-DQBANK-67/USB.NXT
- U801 pad 12: /FPGA-DQBANK-23/USB.DIR -> /FPGA-DQBANK-67/USB.DIR
- U801 pad 13: /FPGA-DQBANK-23/USB.STP -> /FPGA-DQBANK-67/USB.STP
- U801 pad 14: /FPGA-DQBANK-23/USB.CLK -> /FPGA-DQBANK-67/USB.CLK
- U801 pad 17: /FPGA-DQBANK-23/USB.D7 -> /FPGA-DQBANK-67/USB.D7
- U801 pad 18: /FPGA-DQBANK-23/USB.D6 -> /FPGA-DQBANK-67/USB.D6
- U801 pad 19: /FPGA-DQBANK-23/USB.D5 -> /FPGA-DQBANK-67/USB.D5
- U801 pad 20: /FPGA-DQBANK-23/USB.D4 -> /FPGA-DQBANK-67/USB.D4
- U801 pad 21: /FPGA-DQBANK-23/USB.D3 -> /FPGA-DQBANK-67/USB.D3
- U801 pad 22: /FPGA-DQBANK-23/USB.D2 -> /FPGA-DQBANK-67/USB.D2
- U801 pad 23: /FPGA-DQBANK-23/USB.D1 -> /FPGA-DQBANK-67/USB.D1
- U801 pad 24: /FPGA-DQBANK-23/USB.D0 -> /FPGA-DQBANK-67/USB.D0
- U801 pad 9: /FPGA-DQBANK-23/USB.RST -> /FPGA-DQBANK-67/USB.RST
Routing:
- added copper zone on In1.Cu, net GND
- added copper zone on In4.Cu, net GND
Other:
- board outline added: 100 x 100 mm

Commit message: [carrier] connected ethernet, usb and adc to appropriate banks, redpositioned schmitt trigger and USB
Parts:
- removed C1201: 1uF, Capacitor_SMD:C_0805_2012Metric
- removed C609: 0.1uF, Capacitor_SMD:C_0201_0603Metric
- removed C610: 5pF, Capacitor_SMD:C_0603_1608Metric
- removed R817: 2M, Resistor_SMD:R_0603_1608Metric_Pad0.98x0.95mm_HandSolder
- removed R820: 100k, Resistor_SMD:R_0603_1608Metric_Pad0.98x0.95mm_HandSolder
- removed TP803, TP805, TP806: TestPoint, TestPoint:TestPoint_Loop_D1.80mm_Drill1.0mm_Beaded
- added C604: 0.1uF, Capacitor_SMD:C_0201_0603Metric, F.Cu at (14.5, 45.0)
- added C605: 5pF, Capacitor_SMD:C_0603_1608Metric, F.Cu at (11.3, 40.8)
- added C801: 0.1uF, Capacitor_SMD:C_0201_0603Metric, B.Cu at (62.5, 55.6)
- added R802: 3k9, Resistor_SMD:R_0603_1608Metric_Pad0.98x0.95mm_HandSolder, F.Cu at (50.7, 66.9)
- added R803: 100k, Resistor_SMD:R_0603_1608Metric_Pad0.98x0.95mm_HandSolder, F.Cu at (51.6, 69.6)
- added TP801: TestPoint, TestPoint:TestPoint_Loop_D1.80mm_Drill1.0mm_Beaded, F.Cu at (58.8, 56.0)
- added U802: LMV321, Package_TO_SOT_SMD:SOT-23-5, F.Cu at (62.9, 55.6)
- C1202, C1203, C1204, C1205, C1206, C1207, C1208, C1209, C1210, C1211, C1212, C1213, C1214, C1215, C1216, C1217, C1218, C1219, C1220, C1221, C1222, C1223, C1224, C1225, L1201, L1202, L1203: moved to B.Cu
- D801, D802, R813, R821, TP804, TP807, U803, U804: moved to F.Cu
- R811: value 2M -> 100k; moved to F.Cu
- R812: value 100k -> 3k9; moved to F.Cu
- R816: value 6k2 -> 56k; moved to F.Cu
- R818: value 1k2 -> 9k1; moved to F.Cu
- moved R601 293.0 mm to (11.3, 43.3)
- moved Y601 290.6 mm to (15.9, 41.9)
- moved R401 283.1 mm to (114.5, 36.1)
- moved R1213 255.6 mm to (-124.1, 26.7)
- moved R1208 255.6 mm to (-124.0, 28.3)
- moved J201 214.8 mm to (46.1, 179.5)
- moved R1203 207.4 mm to (-125.4, 18.4)
- moved R1204 207.4 mm to (-123.8, 18.6)
- moved R1211 207.4 mm to (-125.3, 21.6)
- moved RN1201 207.4 mm to (-130.4, 19.8)
- moved R1205 207.4 mm to (-127.4, 19.7)
- moved C1229 193.1 mm to (-130.6, 30.1)
- moved D1201 193.1 mm to (-130.6, 27.5)
- moved R1212 193.1 mm to (-129.0, 27.8)
- moved TP1201 193.0 mm to (-133.8, 26.6)
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Connections:
- IC1 pad A11: /ETHERNET-PHY/RGMII_RX.CTL -> /RGMII_RX.CLK
- IC1 pad A12: /ETHERNET-PHY/RGMII_RX.D0 -> /RGMII_TX.CTL
- IC1 pad A13: /ETHERNET-PHY/RGMII_TX.D3 -> unconnected-(IC1C-PT65A-PadA13)
- IC1 pad A14: /ETHERNET-PHY/RGMII_TX.CLK -> unconnected-(IC1C-PT65B-PadA14)
- IC1 pad A15: /ETHERNET-PHY/RGMII_MDIO.CLK -> unconnected-(IC1C-PT67B-PadA15)
- IC1 pad A2: /ANALOG-FRONTEND/ADC.CLK -> unconnected-(IC1B-PT4A-PadA2)
- IC1 pad A3: /ANALOG-FRONTEND/ADC.D1 -> unconnected-(IC1B-PT6A-PadA3)
- IC1 pad A4: /ANALOG-FRONTEND/ADC.D2 -> unconnected-(IC1B-PT6B-PadA4)
- IC1 pad A5: FPGA_ADC_LED1 -> /USB.D3
- IC1 pad A6: FPGA_ADC_LED0 -> /USB.D4
- IC1 pad A7: /CONNECTORS/CON1.T_SCL -> FPGA_CC2
- IC1 pad A8: /CONNECTORS/CON1.T_SDA -> FPGA_USB_SENSE
- IC1 pad B1: unconnected-(IC1G-PL2A/LDQ8-PadB1) -> /ADC.CLK
- IC1 pad B11: unconnected-(IC1C-PT49A-PadB11) -> /RGMII_RX.D0
- IC1 pad B12: /ETHERNET-PHY/RGMII_RX.D1 -> /RGMII_TX.D0
- IC1 pad B13: /ETHERNET-PHY/RGMII_TX.CTL -> /RGMII_TX.CLK
- IC1 pad B14: /ETHERNET-PHY/RGMII_MDIO.DATA -> unconnected-(IC1C-PT67A-PadB14)
- IC1 pad B2: unconnected-(IC1G-PL2B-PadB2) -> /ADC.D0
- IC1 pad B3: /ANALOG-FRONTEND/ADC.D0 -> unconnected-(IC1B-PT4B-PadB3)
- IC1 pad B4: /ANALOG-FRONTEND/ADC.D6 -> /USB.DIR
- IC1 pad B5: /ANALOG-FRONTEND/ADC.OTR -> /USB.D2
- IC1 pad B6: /CONNECTORS/CON1.PWM1 -> unconnected-(IC1B-PT22B-PadB6)
- IC1 pad B7: /CONNECTORS/CON1.B40_EN -> FPGA_CC1
- IC1 pad B8: unconnected-(IC1C-PT35B/PCLKC1_0-PadB8) -> ~{ETH_INT}
- IC1 pad C1: unconnected-(IC1G-PL5A-PadC1) -> /ADC.D3
- IC1 pad C11: unconnected-(IC1C-PT49B-PadC11) -> /RGMII_RX.D1
- IC1 pad C12: /ETHERNET-PHY/RGMII_RX.D2 -> /RGMII_TX.D1
- IC1 pad C13: /ETHERNET-PHY/RGMII_TX.D0 -> /RGMII_MDIO.DATA
- IC1 pad C2: unconnected-(IC1G-PL5B-PadC2) -> /ADC.D4
- IC1 pad C3: unconnected-(IC1G-PL2C-PadC3) -> /ADC.D1
- IC1 pad C4: /ANALOG-FRONTEND/ADC.D5 -> /USB.STP
- IC1 pad C5: /ANALOG-FRONTEND/ADC.D9 -> /USB.D1
- IC1 pad C6: /CONNECTORS/CON1.PWM0 -> /USB.D7
- IC1 pad C7: /CONNECTORS/CON1.S10V_EN -> unconnected-(IC1B-PT27A/PCLKT0_1-PadC7)
- IC1 pad C8: unconnected-(IC1C-PT35A/PCLKT1_0-PadC8) -> Net-(IC1C-PT35A/PCLKT1_0)
- IC1 pad D1: unconnected-(IC1G-PL8A/LDQS8-PadD1) -> /ADC.D7
- IC1 pad D11: unconnected-(IC1C-PT51A-PadD11) -> /RGMII_RX.D2
- IC1 pad D12: /ETHERNET-PHY/RGMII_RX.D3 -> /RGMII_TX.D2
- IC1 pad D13: /ETHERNET-PHY/RGMII_TX.D1 -> /RGMII_MDIO.CLK
- IC1 pad D3: unconnected-(IC1G-PL2D-PadD3) -> /ADC.D2
- IC1 pad D4: /ANALOG-FRONTEND/ADC.D4 -> unconnected-(IC1B-PT9B-PadD4)
- IC1 pad D5: /ANALOG-FRONTEND/ADC.D8 -> /USB.D0
- IC1 pad D6: unconnected-(IC1B-PT20B-PadD6) -> /USB.D6
- IC1 pad D7: /CONNECTORS/CON1.PWM3 -> /USB.CLK
- IC1 pad D9: Net-(IC1C-PT40A) -> unconnected-(IC1C-PT40A-PadD9)
- IC1 pad E10: unconnected-(IC1C-PT47B-PadE10) -> /RGMII_RX.CTL
- IC1 pad E11: unconnected-(IC1C-PT51B-PadE11) -> /RGMII_RX.D3
- IC1 pad E12: /ETHERNET-PHY/RGMII_RX.CLK -> /RGMII_TX.D3
- IC1 pad E13: /ETHERNET-PHY/RGMII_TX.D2 -> unconnected-(IC1C-PT62B-PadE13)
- IC1 pad E2: unconnected-(IC1G-PL8B/LDQSN8-PadE2) -> /ADC.D8
- IC1 pad E3: unconnected-(IC1G-PL5C-PadE3) -> /ADC.D5
- IC1 pad E4: /ANALOG-FRONTEND/ADC.D3 -> /USB.RST
- IC1 pad E5: /ANALOG-FRONTEND/ADC.D7 -> /USB.NXT
- IC1 pad E6: FPGA_ADC_SW -> /USB.D5
- IC1 pad E7: /CONNECTORS/CON1.PWM2 -> unconnected-(IC1B-PT24A/GR_PCLK0_1-PadE7)
- IC1 pad E9: ~{ETH_INT} -> unconnected-(IC1C-PT40B-PadE9)
- IC1 pad F1: unconnected-(IC1G-PL14A/LDQ20-PadF1) -> /CON1.PWM0
- IC1 pad F2: unconnected-(IC1G-PL11C-PadF2) -> FPGA_ADC_SW
- IC1 pad F3: unconnected-(IC1G-PL5D-PadF3) -> /ADC.D6
- IC1 pad F4: unconnected-(IC1G-PL8C-PadF4) -> /ADC.D9
- IC1 pad F5: unconnected-(IC1G-PL8D-PadF5) -> /ADC.OTR
- IC1 pad G2: unconnected-(IC1G-PL14B-PadG2) -> /CON1.PWM1
- IC1 pad G3: unconnected-(IC1G-PL14C-PadG3) -> /CON1.PWM2
- IC1 pad G4: unconnected-(IC1G-PL11B-PadG4) -> FPGA_ADC_LED0
- IC1 pad G5: unconnected-(IC1G-PL11A-PadG5) -> FPGA_ADC_LED1
- IC1 pad H3: unconnected-(IC1G-PL14D-PadH3) -> /CON1.PWM3
- IC1 pad H4: unconnected-(IC1G-PL17B-PadH4) -> /CON1.B40_EN
- IC1 pad H5: unconnected-(IC1G-PL17A-PadH5) -> /CON1.S10V_EN
- IC1 pad J3: Net-(IC1G-PL20C/GR_PCLK7_0) -> unconnected-(IC1G-PL20C/GR_PCLK7_0-PadJ3)
- IC1 pad J4: unconnected-(IC1G-PL17C-PadJ4) -> /CON1.T_SCL
- IC1 pad J5: unconnected-(IC1G-PL17D-PadJ5) -> /CON1.T_SDA
- IC1 pad K4: /FPGA-DQBANK-67/USB.CLK -> Net-(IC1F-PL29A/GR_PCLK6_0)
- IC1 pad L3: /FPGA-DQBANK-67/USB.STP -> unconnected-(IC1F-PL32C-PadL3)
- IC1 pad M3: /FPGA-DQBANK-67/USB.DIR -> unconnected-(IC1F-PL32D-PadM3)
- IC1 pad M4: /FPGA-DQBANK-67/USB.D1 -> unconnected-(IC1F-PL35C-PadM4)
- IC1 pad M5: FPGA_CC1 -> unconnected-(IC1F-PL44C-PadM5)
- IC1 pad N1: /FPGA-DQBANK-67/USB.RST -> unconnected-(IC1F-PL32A/LDQS32-PadN1)
- IC1 pad N3: /FPGA-DQBANK-67/USB.D2 -> unconnected-(IC1F-PL35D-PadN3)
- IC1 pad N4: /FPGA-DQBANK-67/USB.D3 -> unconnected-(IC1F-PL38A/LDQ44-PadN4)
- IC1 pad N5: FPGA_CC2 -> unconnected-(IC1F-PL44D-PadN5)
- IC1 pad P1: /FPGA-DQBANK-67/USB.NXT -> unconnected-(IC1F-PL35A-PadP1)
- IC1 pad P3: /FPGA-DQBANK-67/USB.D4 -> unconnected-(IC1F-PL38B-PadP3)
- IC1 pad P4: FPGA_USB_SENSE -> unconnected-(IC1F-PL41A-PadP4)
- IC1 pad R1: /FPGA-DQBANK-67/USB.D0 -> unconnected-(IC1F-PL35B/VREF1_6-PadR1)
- IC1 pad R2: /FPGA-DQBANK-67/USB.D5 -> unconnected-(IC1F-PL38C-PadR2)
- IC1 pad R5: /FPGA-DQBANK-67/USB.D7 -> unconnected-(IC1F-PL44A/LDQS44-PadR5)
- IC1 pad T2: /FPGA-DQBANK-67/USB.D6 -> unconnected-(IC1F-PL38D-PadT2)
- J901 pad 1: /CONNECTORS/CON1.PWM0 -> /CON1.PWM0
- J901 pad 11: /CONNECTORS/CON1.B40_EN -> /CON1.B40_EN
- J901 pad 13: /CONNECTORS/CON1.T_SCL -> /CON1.T_SCL
- J901 pad 15: /CONNECTORS/CON1.T_SDA -> /CON1.T_SDA
- J901 pad 3: /CONNECTORS/CON1.PWM1 -> /CON1.PWM1
- J901 pad 5: /CONNECTORS/CON1.PWM2 -> /CON1.PWM2
- J901 pad 7: /CONNECTORS/CON1.PWM3 -> /CON1.PWM3
- J901 pad 9: /CONNECTORS/CON1.S10V_EN -> /CON1.S10V_EN
- R1203 pad 2: /ETHERNET-PHY/RGMII_RX.CLK -> /RGMII_RX.CLK
- R1204 pad 1: /ETHERNET-PHY/RGMII_RX.CTL -> /RGMII_RX.CTL
- R1205 pad 1: /ETHERNET-PHY/RGMII_MDIO.DATA -> /RGMII_MDIO.DATA
- R1211 pad 1: /ETHERNET-PHY/RGMII_RX.CLK -> /RGMII_RX.CLK
- R401 pad 1: Net-(IC1C-PT40A) -> Net-(IC1C-PT35A/PCLKT1_0)
- R812 pad 1: /USB-PHY/USB_CC1 -> /USB-PHY/USBCC_VREF_BUFF
- R816 pad 1: /USB-PHY/USB_CC_VREF -> Net-(U802-+)
- R818 pad 2: /USB-PHY/USB_CC_VREF -> Net-(U802-+)
- RN1201 pad 1: /ETHERNET-PHY/RGMII_RX.D0 -> /RGMII_RX.D0
- RN1201 pad 2: /ETHERNET-PHY/RGMII_RX.D1 -> /RGMII_RX.D1
- RN1201 pad 3: /ETHERNET-PHY/RGMII_RX.D2 -> /RGMII_RX.D2
- RN1201 pad 4: /ETHERNET-PHY/RGMII_RX.D3 -> /RGMII_RX.D3
- U1001 pad 10: /ANALOG-FRONTEND/ADC.D7 -> /ADC.D7
- U1001 pad 11: /ANALOG-FRONTEND/ADC.D8 -> /ADC.D8
- U1001 pad 12: /ANALOG-FRONTEND/ADC.D9 -> /ADC.D9
- U1001 pad 13: /ANALOG-FRONTEND/ADC.OTR -> /ADC.OTR
- U1001 pad 15: /ANALOG-FRONTEND/ADC.CLK -> /ADC.CLK
- U1001 pad 3: /ANALOG-FRONTEND/ADC.D0 -> /ADC.D0
- U1001 pad 4: /ANALOG-FRONTEND/ADC.D1 -> /ADC.D1
- U1001 pad 5: /ANALOG-FRONTEND/ADC.D2 -> /ADC.D2
- U1001 pad 6: /ANALOG-FRONTEND/ADC.D3 -> /ADC.D3
- U1001 pad 7: /ANALOG-FRONTEND/ADC.D4 -> /ADC.D4
- U1001 pad 8: /ANALOG-FRONTEND/ADC.D5 -> /ADC.D5
- U1001 pad 9: /ANALOG-FRONTEND/ADC.D6 -> /ADC.D6
- U1201 pad 19: /ETHERNET-PHY/RGMII_TX.D0 -> /RGMII_TX.D0
- U1201 pad 20: /ETHERNET-PHY/RGMII_TX.D1 -> /RGMII_TX.D1
- U1201 pad 21: /ETHERNET-PHY/RGMII_TX.D2 -> /RGMII_TX.D2
- U1201 pad 22: /ETHERNET-PHY/RGMII_TX.D3 -> /RGMII_TX.D3
- U1201 pad 24: /ETHERNET-PHY/RGMII_TX.CLK -> /RGMII_TX.CLK
- U1201 pad 25: /ETHERNET-PHY/RGMII_TX.CTL -> /RGMII_TX.CTL
- U1201 pad 27: /ETHERNET-PHY/RGMII_RX.D3 -> /RGMII_RX.D3
- U1201 pad 28: /ETHERNET-PHY/RGMII_RX.D2 -> /RGMII_RX.D2
- U1201 pad 31: /ETHERNET-PHY/RGMII_RX.D1 -> /RGMII_RX.D1
- U1201 pad 32: /ETHERNET-PHY/RGMII_RX.D0 -> /RGMII_RX.D0
- U1201 pad 33: /ETHERNET-PHY/RGMII_RX.CTL -> /RGMII_RX.CTL
- U1201 pad 35: /ETHERNET-PHY/RGMII_RX.CLK -> /RGMII_RX.CLK
- U1201 pad 36: /ETHERNET-PHY/RGMII_MDIO.CLK -> /RGMII_MDIO.CLK
- U1201 pad 37: /ETHERNET-PHY/RGMII_MDIO.DATA -> /RGMII_MDIO.DATA
- U801 pad 11: /FPGA-DQBANK-67/USB.NXT -> /USB.NXT
- U801 pad 12: /FPGA-DQBANK-67/USB.DIR -> /USB.DIR
- U801 pad 13: /FPGA-DQBANK-67/USB.STP -> /USB.STP
- U801 pad 14: /FPGA-DQBANK-67/USB.CLK -> /USB.CLK
- U801 pad 17: /FPGA-DQBANK-67/USB.D7 -> /USB.D7
- U801 pad 18: /FPGA-DQBANK-67/USB.D6 -> /USB.D6
- U801 pad 19: /FPGA-DQBANK-67/USB.D5 -> /USB.D5
- U801 pad 20: /FPGA-DQBANK-67/USB.D4 -> /USB.D4
- U801 pad 21: /FPGA-DQBANK-67/USB.D3 -> /USB.D3
- U801 pad 22: /FPGA-DQBANK-67/USB.D2 -> /USB.D2
- U801 pad 23: /FPGA-DQBANK-67/USB.D1 -> /USB.D1
- U801 pad 24: /FPGA-DQBANK-67/USB.D0 -> /USB.D0
- U801 pad 9: /FPGA-DQBANK-67/USB.RST -> /USB.RST
- U803 pad 4: /USB-PHY/USB_CC_VREF -> /USB-PHY/USB_CC2
- U804 pad 4: /USB-PHY/USB_CC_VREF -> /USB-PHY/USB_CC1
- Y601 pad 3: Net-(IC1G-PL20C/GR_PCLK7_0) -> Net-(IC1F-PL29A/GR_PCLK6_0)
Other:
- board size 100 x 100 mm -> 82.8 x 100 mm
