File: acoustic-carrier-hw/acoustic-carrier-board/acoustic-carrier-board.kicad_pcb (KiCad board)
At the start: 6 copper layers, 82.8 x 100 mm, 359 parts, among them IC1 ECP5-BGA256, IC1101 MT41K256M16TW-107_P, J1001 BWU.FL-IPEX1, J1002 BWU.FL-IPEX1, J1003 BWU.FL-IPEX1, J1004 BWU.FL-IPEX1, J1005 BWU.FL-IPEX1, J1006 BWU.FL-IPEX1, J1007 8P8C_Shielded, J1008 BWU.FL-IPEX1, J1201 HR911130A, J201 Conn_02x08_Odd_Even, J701 Conn_01x10_Socket, J702 Conn_01x08_Socket, J801 TYPE-C-31-M-12, J901 Conn_02x08_Odd_Even, Q201 AO3401A, U1001 MS9280, U1002 THS4521IDGK, U1003 DGQ2788AEN-T1-GE4, U1004 LMV321, U1005 TL432DBZ, U1201 KSZ9031RN, U201 TPS2121RUX, U202 TLV62569DBV, U203 TLV62569DBV, U204 TLV62569DBV, U205 TLV62569DBV, U206 OPA376xxDBV, U701 W25Q128JVS, U702 W25Q128JVS, U801 USB3300-EZK, U802 LMV321, Y1201 25MHz, Y601 Crystal Oscillator, Y801 Crystal_GND24_Small

Commit message: [¢arrier] Placed decoupling for some banks, placed dc-dc converterss (next) switch dc-dc converter pins around, switch adc-inputs around
Parts:
- removed C604: 0.1uF, Capacitor_SMD:C_0201_0603Metric
- removed C605: 5pF, Capacitor_SMD:C_0603_1608Metric
- removed R601: 1k, Resistor_SMD:R_0603_1608Metric
- removed Y601: Crystal Oscillator, Crystal:Crystal_SMD_3225-4Pin_3.2x2.5mm
- added C1022: 10nF, Capacitor_SMD:C_0201_0603Metric, B.Cu at (195.5, 103.4)
- added C225: 0.1uF, Capacitor_SMD:C_0201_0603Metric, B.Cu at (98.8, 106.4)
- added C226: 10nF, Capacitor_SMD:C_0201_0603Metric, B.Cu at (102.1, 105.2)
- added C606: 0.1uF, Capacitor_SMD:C_0201_0603Metric, B.Cu at (76.0, 87.0)
- added C607: 5pF, Capacitor_SMD:C_0603_1608Metric, F.Cu at (79.3, 87.3)
- added C802: 10nF, Capacitor_SMD:C_0201_0603Metric, B.Cu at (61.4, 55.1)
- added R602: 1k, Resistor_SMD:R_0603_1608Metric, F.Cu at (73.5, 87.6)
- added Y602: Crystal Oscillator, Crystal:Crystal_SMD_3225-4Pin_3.2x2.5mm, F.Cu at (76.4, 87.6)
- C1001, C1002, C1003, C1004, C1005, C1006, C1007, C1008, C1013, C1014, C1021, C204, C205, C206, C207, C208, C210, C211, C212, C213, C214, C215, C216, C218, C220, C221, C222, C223, C224, C404, C405, C406, JP1001, JP1002, JP1003, JP1006, JP1007, JP1008, L1001, R1030, R1031, R224: moved to B.Cu
- moved TP209 474.2 mm to (51.4, 121.9)
- moved L204 468.9 mm to (48.5, 117.7)
- moved C223 467.3 mm to (52.7, 117.5)
- moved R225 464.8 mm to (52.5, 112.2), turned to 180 degrees
- moved U205 463.6 mm to (48.7, 113.6)
- moved R218 459.7 mm to (52.5, 114.6), turned to -90 degrees
- moved C220 451.0 mm to (51.5, 114.9), turned to 90 degrees
- moved C221 450.9 mm to (51.1, 119.3)
- moved C222 450.7 mm to (53.0, 114.9), turned to 90 degrees
- moved C224 450.1 mm to (47.6, 113.1), turned to -90 degrees
- moved R217 446.3 mm to (52.8, 117.5)
- moved C219 445.5 mm to (51.3, 115.0), turned to 90 degrees
- moved TP208 438.3 mm to (103.5, 100.3), turned to 90 degrees
- moved R222 434.3 mm to (99.3, 102.6), turned to -90 degrees
- moved R224 433.4 mm to (100.9, 106.4), turned to -90 degrees
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Connections:
- net Net-(IC1A-VCCAUX_1) renamed /FPGA-POWER/VAUX
- IC1 pad B1: /ADC.CLK -> unconnected-(IC1G-PL2A/LDQ8-PadB1)
- IC1 pad B2: /ADC.D0 -> unconnected-(IC1G-PL2B-PadB2)
- IC1 pad C1: /ADC.D3 -> Net-(IC1G-PL5A)
- IC1 pad C2: /ADC.D4 -> unconnected-(IC1G-PL5B-PadC2)
- IC1 pad C3: /ADC.D1 -> unconnected-(IC1G-PL2C-PadC3)
- IC1 pad D1: /ADC.D7 -> unconnected-(IC1G-PL8A/LDQS8-PadD1)
- IC1 pad D3: /ADC.D2 -> unconnected-(IC1G-PL2D-PadD3)
- IC1 pad E2: /ADC.D8 -> unconnected-(IC1G-PL8B/LDQSN8-PadE2)
- IC1 pad E3: /ADC.D5 -> unconnected-(IC1G-PL5C-PadE3)
- IC1 pad F1: /CON1.PWM0 -> unconnected-(IC1G-PL14A/LDQ20-PadF1)
- IC1 pad F2: FPGA_ADC_SW -> unconnected-(IC1G-PL11C-PadF2)
- IC1 pad F3: /ADC.D6 -> unconnected-(IC1G-PL5D-PadF3)
- IC1 pad F4: /ADC.D9 -> unconnected-(IC1G-PL8C-PadF4)
- IC1 pad F5: /ADC.OTR -> unconnected-(IC1G-PL8D-PadF5)
- IC1 pad G2: /CON1.PWM1 -> unconnected-(IC1G-PL14B-PadG2)
- IC1 pad G3: /CON1.PWM2 -> unconnected-(IC1G-PL14C-PadG3)
- IC1 pad G4: FPGA_ADC_LED0 -> unconnected-(IC1G-PL11B-PadG4)
- IC1 pad G5: FPGA_ADC_LED1 -> unconnected-(IC1G-PL11A-PadG5)
- IC1 pad H3: /CON1.PWM3 -> unconnected-(IC1G-PL14D-PadH3)
- IC1 pad H4: /CON1.B40_EN -> unconnected-(IC1G-PL17B-PadH4)
- IC1 pad H5: /CON1.S10V_EN -> unconnected-(IC1G-PL17A-PadH5)
- IC1 pad J4: /CON1.T_SCL -> unconnected-(IC1G-PL17C-PadJ4)
- IC1 pad J5: /CON1.T_SDA -> unconnected-(IC1G-PL17D-PadJ5)
- IC1 pad K4: Net-(IC1F-PL29A/GR_PCLK6_0) -> /ADC.D3
- IC1 pad K5: unconnected-(IC1F-PL29B-PadK5) -> /ADC.D4
- IC1 pad L1: unconnected-(IC1F-PL26A/LDQ32/PCLKT6_1-PadL1) -> /ADC.CLK
- IC1 pad L2: unconnected-(IC1F-PL26B/PCLKC6_1-PadL2) -> /ADC.D0
- IC1 pad L3: unconnected-(IC1F-PL32C-PadL3) -> /ADC.D9
- IC1 pad L4: unconnected-(IC1F-PL29C/PL29C-PadL4) -> /ADC.D5
- IC1 pad L5: unconnected-(IC1F-PL29D-PadL5) -> /ADC.D6
- IC1 pad M1: unconnected-(IC1F-PL26C/PCLKT6_0-PadM1) -> /ADC.D1
- IC1 pad M2: unconnected-(IC1F-PL26D/PCLKC6_0-PadM2) -> /ADC.D2
- IC1 pad M3: unconnected-(IC1F-PL32D-PadM3) -> /ADC.OTR
- IC1 pad M4: unconnected-(IC1F-PL35C-PadM4) -> FPGA_ADC_SW
- IC1 pad M5: unconnected-(IC1F-PL44C-PadM5) -> /CON1.T_SCL
- IC1 pad N1: unconnected-(IC1F-PL32A/LDQS32-PadN1) -> /ADC.D7
- IC1 pad N4: unconnected-(IC1F-PL38A/LDQ44-PadN4) -> /CON1.PWM0
- IC1 pad N5: unconnected-(IC1F-PL44D-PadN5) -> /CON1.T_SDA
- IC1 pad P1: unconnected-(IC1F-PL35A-PadP1) -> FPGA_ADC_LED1
- IC1 pad P2: unconnected-(IC1F-PL32B/LDQSN32-PadP2) -> /ADC.D8
- IC1 pad P3: unconnected-(IC1F-PL38B-PadP3) -> /CON1.PWM1
- IC1 pad R1: unconnected-(IC1F-PL35B/VREF1_6-PadR1) -> FPGA_ADC_LED0
- IC1 pad R2: unconnected-(IC1F-PL38C-PadR2) -> /CON1.PWM2
- IC1 pad R5: unconnected-(IC1F-PL44A/LDQS44-PadR5) -> /CON1.S10V_EN
- IC1 pad T2: unconnected-(IC1F-PL38D-PadT2) -> /CON1.PWM3
- IC1 pad T4: unconnected-(IC1F-PL44B/LDQSN44-PadT4) -> /CON1.B40_EN
Other:
- board size 82.8 x 100 mm -> 100 x 100 mm

Commit message: [carrier] Rearanged big parts of the analog PCB
Parts:
- removed C1009: 10uF, Capacitor_SMD:C_0603_1608Metric
- removed C1010: 0.1uF, Capacitor_SMD:C_0201_0603Metric
- removed C1011: 10nF, Capacitor_SMD:C_0201_0603Metric
- removed R1008: 0, Resistor_SMD:R_0603_1608Metric
- removed R201: 24k, Resistor_SMD:R_0603_1608Metric
- removed R202: 5.1k, Resistor_SMD:R_0603_1608Metric
- removed TP1002, TP1003, TP201: TestPoint, TestPoint:TestPoint_Loop_D1.80mm_Drill1.0mm_Beaded
- removed TP204: TestPoint, TestPoint:TestPoint_Pad_1.0x1.0mm
- added C1023: 10uF, Capacitor_SMD:C_0603_1608Metric, B.Cu at (97.3, 123.6)
- added C1024: 0.1uF, Capacitor_SMD:C_0201_0603Metric, B.Cu at (95.1, 124.1)
- added C1025: 10nF, Capacitor_SMD:C_0201_0603Metric, B.Cu at (95.1, 123.4)
- added J1009: BWU.FL-IPEX1, iw-connector:BWU.FL-IPEX1, B.Cu at (65.3, 136.2)
- added J1010: BWU.FL-IPEX1, iw-connector:BWU.FL-IPEX1, B.Cu at (72.2, 130.5)
- added R1039: 0, Resistor_SMD:R_0603_1608Metric, B.Cu at (76.4, 135.7)
- added R226: 24k, Resistor_SMD:R_0603_1608Metric, B.Cu at (44.3, 77.8)
- added R227: 5.1k, Resistor_SMD:R_0603_1608Metric, B.Cu at (45.8, 77.8)
- added TP210: TestPoint, TestPoint:TestPoint_Loop_D1.80mm_Drill1.0mm_Beaded, F.Cu at (62.7, 60.1)
- C202: value 1uF -> 0.1uF; footprint Capacitor_SMD:C_0805_2012Metric -> Capacitor_SMD:C_0201_0603Metric; moved to B.Cu
- J1003, J1004, J1005, R1006, R1028, R203, R204, R205, R207, TP1008: moved to B.Cu
- R1012, R1017, R1018, R1020: footprint Resistor_SMD:R_0603_1608Metric -> Resistor_SMD:R_0402_1005Metric_Pad0.72x0.64mm_HandSolder
- R1015: footprint Resistor_SMD:R_0603_1608Metric -> Resistor_SMD:R_0402_1005Metric_Pad0.72x0.64mm_HandSolder; moved to B.Cu
- moved RJ1001 72.8 mm to (75.6, 141.0)
- moved J1007 72.1 mm to (112.8, 138.5), turned to 90 degrees
- moved C1017 66.4 mm to (106.3, 133.4), turned to 180 degrees
- moved C1018 65.0 mm to (106.3, 135.0), turned to 180 degrees
- moved R1027 62.3 mm to (103.9, 132.7), turned to -90 degrees
- moved R1029 59.3 mm to (103.8, 135.7), turned to -90 degrees
- moved R1012 49.8 mm to (94.8, 129.8), turned to 90 degrees
- moved R1018 47.3 mm to (92.9, 129.8)
- moved TP1008 47.2 mm to (96.3, 134.6), turned to 0 degrees
- moved C1021 44.5 mm to (94.1, 132.8), turned to 180 degrees
- moved U1003 44.4 mm to (93.8, 132.6), turned to 0 degrees
- moved C301 42.5 mm to (-0.31, 224.3)
- moved C302 42.5 mm to (-1.81, 224.3)
- moved C303 42.5 mm to (-2.56, 224.4)
- moved C305 42.5 mm to (-3.36, 224.3)
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Connections:
- C1012 pad 2: Net-(U1002-+) -> Net-(U1002--)
- C1016 pad 1: Net-(U1002--) -> Net-(U1002-+)
- C1017 pad 2: /ANALOG-FRONTEND/RJ45_ADC_AIN+ -> /ANALOG-FRONTEND/RJ45_ADC_AIN-
- C1018 pad 2: /ANALOG-FRONTEND/RJ45_ADC_AIN- -> /ANALOG-FRONTEND/RJ45_ADC_AIN+
- IC1 pad K4: /ADC.D3 -> /CON1.S10V_EN
- IC1 pad K5: /ADC.D4 -> /CON1.B40_EN
- IC1 pad L1: /ADC.CLK -> /CON1.PWM0
- IC1 pad L2: /ADC.D0 -> /CON1.PWM1
- IC1 pad L3: /ADC.D9 -> unconnected-(IC1F-PL32C-PadL3)
- IC1 pad L4: /ADC.D5 -> /CON1.T_SCL
- IC1 pad L5: /ADC.D6 -> /CON1.T_SDA
- IC1 pad M1: /ADC.D1 -> /CON1.PWM2
- IC1 pad M2: /ADC.D2 -> /CON1.PWM3
- IC1 pad M3: /ADC.OTR -> unconnected-(IC1F-PL32D-PadM3)
- IC1 pad M4: FPGA_ADC_SW -> unconnected-(IC1F-PL35C-PadM4)
- IC1 pad M5: /CON1.T_SCL -> /ADC.D8
- IC1 pad M6: unconnected-(IC1F-PL47A-PadM6) -> /ADC.D2
- IC1 pad N1: /ADC.D7 -> unconnected-(IC1F-PL32A/LDQS32-PadN1)
- IC1 pad N4: /CON1.PWM0 -> unconnected-(IC1F-PL38A/LDQ44-PadN4)
- IC1 pad N5: /CON1.T_SDA -> /ADC.D7
- IC1 pad N6: unconnected-(IC1F-PL47B-PadN6) -> /ADC.D1
- IC1 pad P1: FPGA_ADC_LED1 -> unconnected-(IC1F-PL35A-PadP1)
- IC1 pad P2: /ADC.D8 -> unconnected-(IC1F-PL32B/LDQSN32-PadP2)
- IC1 pad P3: /CON1.PWM1 -> FPGA_ADC_LED1
- IC1 pad P4: unconnected-(IC1F-PL41A-PadP4) -> /ADC.D6
- IC1 pad P5: unconnected-(IC1F-PL47D/LLC_GPLL0C_IN-PadP5) -> /ADC.D0
- IC1 pad P6: unconnected-(IC1F-PL47C/LLC_GPLL0T_IN-PadP6) -> /ADC.CLK
- IC1 pad R1: FPGA_ADC_LED0 -> unconnected-(IC1F-PL35B/VREF1_6-PadR1)
- IC1 pad R2: /CON1.PWM2 -> FPGA_ADC_LED0
- IC1 pad R3: unconnected-(IC1F-PL41B-PadR3) -> /ADC.D5
- IC1 pad R4: unconnected-(IC1F-PL41C-PadR4) -> /ADC.D4
- IC1 pad R5: /CON1.S10V_EN -> /ADC.OTR
- IC1 pad T2: /CON1.PWM3 -> FPGA_ADC_SW
- IC1 pad T3: unconnected-(IC1F-PL41D-PadT3) -> /ADC.D3
- IC1 pad T4: /CON1.B40_EN -> /ADC.D9
- R1009 pad 2: Net-(U1002-+) -> Net-(U1002--)
- R1012 pad 1: Net-(R1007-Pad2) -> Net-(U1003-COM1)
- R1012 pad 2: Net-(U1003-COM1) -> Net-(R1007-Pad2)
- R1013 pad 1: Net-(U1002-+) -> Net-(U1002--)
- R1015 pad 1: Net-(U1002-~{PD}) -> VCORE_3V3
- R1015 pad 2: VCORE_3V3 -> Net-(U1002-~{PD})
- R1017 pad 1: /ANALOG-FRONTEND/ADC_AIN+ -> Net-(R1009-Pad1)
- R1017 pad 2: Net-(R1009-Pad1) -> /ANALOG-FRONTEND/ADC_AIN+
- R1018 pad 1: Net-(R1018-Pad1) -> Net-(U1003-COM2)
- R1018 pad 2: Net-(U1003-COM2) -> Net-(R1018-Pad2)
- R1020 pad 1: /ANALOG-FRONTEND/ADC_AIN- -> Net-(R1019-Pad1)
- R1020 pad 2: Net-(R1019-Pad1) -> /ANALOG-FRONTEND/ADC_AIN-
- R1021 pad 1: Net-(U1002--) -> Net-(U1002-+)
- R1021 pad 2: Net-(R1018-Pad1) -> Net-(R1018-Pad2)
- R1024 pad 1: Net-(U1002--) -> Net-(U1002-+)
- R1026 pad 1: Net-(R1018-Pad1) -> Net-(R1018-Pad2)
- R1027 pad 2: /ANALOG-FRONTEND/RJ45_ADC_AIN+ -> /ANALOG-FRONTEND/RJ45_ADC_AIN-
- R1029 pad 1: /ANALOG-FRONTEND/RJ45_ADC_AIN- -> /ANALOG-FRONTEND/RJ45_ADC_AIN+
- R203 pad 2: Net-(U201-OV2) -> Net-(U201-OV1)
- R207 pad 1: Net-(U201-OV2) -> Net-(U201-OV1)
- RJ1001 pad 1: /ANALOG-FRONTEND/MAG_ADC_AIN+ -> Net-(J1009-In)
- RJ1001 pad 2: /ANALOG-FRONTEND/MAG_ADC_AIN- -> Net-(J1010-In)
- RJ1001 pad 3: Net-(RJ1001-Pad3) -> /ANALOG-FRONTEND/MAG_ADC_AIN-
- RJ1001 pad 4: Net-(R1008-Pad2) -> GND
- RJ1001 pad 5: GND -> Net-(R1039-Pad2)
- RJ1001 pad 6: Net-(RJ1001-Pad6) -> /ANALOG-FRONTEND/MAG_ADC_AIN+
- U1002 pad 4: Net-(C1016-Pad2) -> Net-(C1012-Pad1)
- U1002 pad 5: Net-(C1012-Pad1) -> Net-(C1016-Pad2)
- U1003 pad 1: /ANALOG-FRONTEND/MAG_ADC_AIN- -> /ANALOG-FRONTEND/MAG_ADC_AIN+
- U1003 pad 11: /ANALOG-FRONTEND/RJ45_ADC_AIN+ -> /ANALOG-FRONTEND/RJ45_ADC_AIN-
- U1003 pad 13: /ANALOG-FRONTEND/MAG_ADC_AIN+ -> /ANALOG-FRONTEND/MAG_ADC_AIN-
- U1003 pad 15: /ANALOG-FRONTEND/RJ45_ADC_AIN- -> /ANALOG-FRONTEND/RJ45_ADC_AIN+
- U201 pad 2: Net-(Q201-D) -> /POWER/USB_VBUS
- U201 pad 7: /POWER/USB_VBUS -> Net-(Q201-D)

Commit message: [¢arrier] Placed power supply circuitry appropraitely, changed power connector (next) Place schmitt triggers between usb and power, put critical circuitry closer together, place config circuitry
Parts:
- removed C606: 0.1uF, Capacitor_SMD:C_0201_0603Metric
- removed C607: 5pF, Capacitor_SMD:C_0603_1608Metric
- removed J201: Conn_02x08_Odd_Even, Connector_PinSocket_2.54mm:PinSocket_2x08_P2.54mm_Horizontal
- removed R214: 0, Resistor_SMD:R_0805_2012Metric_Pad1.20x1.40mm_HandSolder
- removed R602: 1k, Resistor_SMD:R_0603_1608Metric
- removed Y602: Crystal Oscillator, Crystal:Crystal_SMD_3225-4Pin_3.2x2.5mm
- added C407: 0.1uF, Capacitor_SMD:C_0201_0603Metric, F.Cu at (219.5, 60.9)
- added C408: 5pF, Capacitor_SMD:C_0603_1608Metric, F.Cu at (216.3, 56.8)
- added J202: Conn_02x04_Odd_Even, Connector_PinSocket_2.54mm:PinSocket_2x04_P2.54mm_Horizontal, F.Cu at (122.0, 56.7)
- added R601: 0, Resistor_SMD:R_0603_1608Metric, F.Cu at (216.3, 65.0)
- added Y401: Crystal Oscillator, Crystal:Crystal_SMD_3225-4Pin_3.2x2.5mm, F.Cu at (220.9, 57.8)
- C201, C310, C311, C312, C313, L301: moved to B.Cu
- R401: value 0 -> 1k
- moved L301 187.7 mm to (78.1, 69.0), turned to 90 degrees
- moved C313 179.0 mm to (85.8, 83.0), turned to 90 degrees
- moved C312 178.6 mm to (87.0, 83.0), turned to 90 degrees
- moved C311 173.3 mm to (89.8, 89.7), turned to 180 degrees
- moved C310 169.9 mm to (86.9, 92.5), turned to 90 degrees
- moved TP205 169.3 mm to (136.2, -37.1)
- moved TP207 166.2 mm to (135.6, -41.7)
- moved C804 126.2 mm to (166.6, 25.3), turned to 180 degrees
- moved U803 124.5 mm to (166.0, 26.4), turned to 90 degrees
- moved C808 124.4 mm to (165.1, 25.9), turned to -90 degrees
- moved C817 124.0 mm to (166.5, 27.1), turned to 180 degrees
- moved R812 123.8 mm to (168.6, 28.6), turned to -90 degrees
- moved R813 122.1 mm to (163.5, 26.9), turned to 90 degrees
- moved R815 122.0 mm to (163.4, 26.9), turned to 90 degrees
- moved R811 120.8 mm to (166.0, 29.5), turned to 180 degrees
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Connections:
- IC1 pad A11: /RGMII_RX.CLK -> /USB.D1
- IC1 pad A12: /RGMII_TX.CTL -> /USB.D2
- IC1 pad A14: unconnected-(IC1C-PT65B-PadA14) -> FPGA_CC1
- IC1 pad A15: unconnected-(IC1C-PT67B-PadA15) -> FPGA_USB_SENSE
- IC1 pad A5: /USB.D3 -> unconnected-(IC1B-PT18A-PadA5)
- IC1 pad A6: /USB.D4 -> unconnected-(IC1B-PT18B-PadA6)
- IC1 pad A7: FPGA_CC2 -> unconnected-(IC1B-PT29A/PCLKT0_0-PadA7)
- IC1 pad A8: FPGA_USB_SENSE -> unconnected-(IC1B-PT29B/PCLKC0_0-PadA8)
- IC1 pad B11: /RGMII_RX.D0 -> /USB.STP
- IC1 pad B12: /RGMII_TX.D0 -> /USB.D3
- IC1 pad B13: /RGMII_TX.CLK -> /USB.D7
- IC1 pad B14: unconnected-(IC1C-PT67A-PadB14) -> FPGA_CC2
- IC1 pad B4: /USB.DIR -> unconnected-(IC1B-PT11B-PadB4)
- IC1 pad B5: /USB.D2 -> unconnected-(IC1B-PT15B-PadB5)
- IC1 pad B7: FPGA_CC1 -> unconnected-(IC1B-PT27B/PCLKC0_1-PadB7)
- IC1 pad B8: ~{ETH_INT} -> unconnected-(IC1C-PT35B/PCLKC1_0-PadB8)
- IC1 pad C1: Net-(IC1G-PL5A) -> unconnected-(IC1G-PL5A-PadC1)
- IC1 pad C11: /RGMII_RX.D1 -> /USB.DIR
- IC1 pad C12: /RGMII_TX.D1 -> /USB.D4
- IC1 pad C13: /RGMII_MDIO.DATA -> unconnected-(IC1C-PT60B-PadC13)
- IC1 pad C4: /USB.STP -> unconnected-(IC1B-PT11A-PadC4)
- IC1 pad C5: /USB.D1 -> unconnected-(IC1B-PT15A-PadC5)
- IC1 pad C6: /USB.D7 -> unconnected-(IC1B-PT22A-PadC6)
- IC1 pad C8: Net-(IC1C-PT35A/PCLKT1_0) -> unconnected-(IC1C-PT35A/PCLKT1_0-PadC8)
- IC1 pad C9: ETH_REFCLK -> unconnected-(IC1C-PT38B/GR_PCLK1_1-PadC9)
- IC1 pad D1: unconnected-(IC1G-PL8A/LDQS8-PadD1) -> /RGMII_RX.D0
- IC1 pad D10: unconnected-(IC1C-PT47A-PadD10) -> /USB.RST
- IC1 pad D11: /RGMII_RX.D2 -> /USB.NXT
- IC1 pad D12: /RGMII_TX.D2 -> /USB.D5
- IC1 pad D13: /RGMII_MDIO.CLK -> unconnected-(IC1C-PT62A-PadD13)
- IC1 pad D5: /USB.D0 -> unconnected-(IC1B-PT13B-PadD5)
- IC1 pad D6: /USB.D6 -> unconnected-(IC1B-PT20B-PadD6)
- IC1 pad D7: /USB.CLK -> unconnected-(IC1B-PT24B/GR_PCLK0_0-PadD7)
- IC1 pad E1: unconnected-(IC1G-PL11D/LDQ8-PadE1) -> /RGMII_TX.D1
- IC1 pad E10: /RGMII_RX.CTL -> unconnected-(IC1C-PT47B-PadE10)
- IC1 pad E11: /RGMII_RX.D3 -> /USB.D0
- IC1 pad E12: /RGMII_TX.D3 -> /USB.D6
- IC1 pad E13: unconnected-(IC1C-PT62B-PadE13) -> /USB.CLK
- IC1 pad E2: unconnected-(IC1G-PL8B/LDQSN8-PadE2) -> /RGMII_RX.D1
- IC1 pad E4: /USB.RST -> unconnected-(IC1B-PT9A-PadE4)
- IC1 pad E5: /USB.NXT -> unconnected-(IC1B-PT13A-PadE5)
- IC1 pad E6: /USB.D5 -> unconnected-(IC1B-PT20A-PadE6)
- IC1 pad E7: unconnected-(IC1B-PT24A/GR_PCLK0_1-PadE7) -> Net-(IC1B-PT24A/GR_PCLK0_1)
- IC1 pad F1: unconnected-(IC1G-PL14A/LDQ20-PadF1) -> /RGMII_TX.D2
- IC1 pad F2: unconnected-(IC1G-PL11C-PadF2) -> /RGMII_TX.D0
- IC1 pad F3: unconnected-(IC1G-PL5D-PadF3) -> /RGMII_RX.CTL
- IC1 pad F4: unconnected-(IC1G-PL8C-PadF4) -> /RGMII_RX.D2
- IC1 pad F5: unconnected-(IC1G-PL8D-PadF5) -> /RGMII_RX.D3
- IC1 pad G2: unconnected-(IC1G-PL14B-PadG2) -> /RGMII_TX.D3
- IC1 pad G3: unconnected-(IC1G-PL14C-PadG3) -> /RGMII_TX.CLK
- IC1 pad G4: unconnected-(IC1G-PL11B-PadG4) -> /RGMII_TX.CTL
- IC1 pad G5: unconnected-(IC1G-PL11A-PadG5) -> /RGMII_RX.CLK
- IC1 pad H3: unconnected-(IC1G-PL14D-PadH3) -> /RGMII_MDIO.DATA
- IC1 pad H5: unconnected-(IC1G-PL17A-PadH5) -> /RGMII_MDIO.CLK
- IC1 pad J2: unconnected-(IC1G-PL23B/PCLKC7_1-PadJ2) -> Net-(IC1G-PL23B/PCLKC7_1)
- IC1 pad J3: unconnected-(IC1G-PL20C/GR_PCLK7_0-PadJ3) -> ETH_REFCLK
- IC1 pad K1: unconnected-(IC1G-PL23C/PCLKT7_0-PadK1) -> ~{ETH_INT}
- L301 pad 2: VAUX_2V5 -> +2V5
- R401 pad 1: Net-(IC1C-PT35A/PCLKT1_0) -> VCORE_3V3
- R401 pad 2: ~{ETH_RESET} -> Net-(Y401-Tri-State)
Other:
- board size 100 x 100 mm -> 78.8 x 95 mm
