File: acoustic-carrier-hw/acoustic-carrier-board/fpga-power.kicad_sch (KiCad schematic)
At the start: 15 parts, among them IC1 ECP5-BGA256

Commit message: [carrier] Removed USB-switch, placed decouplpling for DDR3 and ECP5U (next) consider adding buffers on CC1 and CC2 pins
Parts:
- C301, C302, C303, C304, C305, C306, C310, C311: footprint Capacitor_SMD:C_0402_1005Metric -> Capacitor_SMD:C_0201_0603Metric; LPN C307331 -> C22435929; MPN CL05B104KB54PNC -> CGA0201X7R104K160ET
Changed lines of the file:
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@@
 			)
 		)
-		(property "Footprint" "Capacitor_SMD:C_0402_1005Metric"
+		(property "Footprint" "Capacitor_SMD:C_0201_0603Metric"
 			(at 144.78 64.77 0)
 			(effects
@@
 			)
 		)
-		(property "Datasheet" "~"
+		(property "Datasheet" "https://jlcpcb.com/api/file/downloadByFileSystemAccessId/8603345729432014848"
 			(at 144.78 64.77 0)
 			(effects
@@
 			)
 		)
-		(property "LPN" "C307331"
+		(property "LPN" "C22435929"
 			(at 144.78 64.77 0)
 			(effects
@@
 			)
 		)
-		(property "MPN" "CL05B104KB54PNC"
+		(property "MPN" "CGA0201X7R104K160ET "
 			(at 144.78 64.77 0)
 			(effects
@@
 			)
 		)
-		(property "Footprint" "Capacitor_SMD:C_0402_1005Metric"
+		(property "Footprint" "Capacitor_SMD:C_0201_0603Metric"
 			(at 151.13 128.27 0)
 			(effects
@@
 			)
 		)
-		(property "Datasheet" "~"
+		(property "Datasheet" "https://jlcpcb.com/api/file/downloadByFileSystemAccessId/8603345729432014848"
 			(at 151.13 128.27 0)
 			(effects
@@
 			)
 		)
-		(property "LPN" "C307331"
+		(property "LPN" "C22435929"
 			(at 151.13 128.27 0)
 			(effects
@@
 			)
 		)
-		(property "MPN" "CL05B104KB54PNC"
+		(property "MPN" "CGA0201X7R104K160ET "
 			(at 151.13 128.27 0)
 			(effects
@@
 			)
 		)
-		(property "Footprint" "Capacitor_SMD:C_0402_1005Metric"
+		(property "Footprint" "Capacitor_SMD:C_0201_0603Metric"
 			(at 123.19 64.77 0)
 			(effects
@@
 			)
 		)
-		(property "Datasheet" "~"
+		(property "Datasheet" "https://jlcpcb.com/api/file/downloadByFileSystemAccessId/8603345729432014848"
 			(at 123.19 64.77 0)
 			(effects
@@
 			)
 		)
-		(property "LPN" "C307331"
+		(property "LPN" "C22435929"
 			(at 123.19 64.77 0)
 			(effects
@@
 			)
 		)
-		(property "MPN" "CL05B104KB54PNC"
+		(property "MPN" "CGA0201X7R104K160ET "
 			(at 123.19 64.77 0)
 			(effects
@@
 			)
 		)
-		(property "Footprint" "Capacitor_SMD:C_0402_1005Metric"
+		(property "Footprint" "Capacitor_SMD:C_0201_0603Metric"
 			(at 151.13 64.77 0)
 			(effects
@@
 			)
 		)
-		(property "Datasheet" "~"
+		(property "Datasheet" "https://jlcpcb.com/api/file/downloadByFileSystemAccessId/8603345729432014848"
 			(at 151.13 64.77 0)
 			(effects
@@
 			)
 		)
-		(property "LPN" "C307331"
+		(property "LPN" "C22435929"
 			(at 151.13 64.77 0)
 			(effects
@@
 			)
 		)
-		(property "MPN" "CL05B104KB54PNC"
+		(property "MPN" "CGA0201X7R104K160ET "
 			(at 151.13 64.77 0)
 			(effects
@@
 			)
 		)
-		(property "Footprint" "Capacitor_SMD:C_0402_1005Metric"
+		(property "Footprint" "Capacitor_SMD:C_0201_0603Metric"
 			(at 138.43 64.77 0)
 			(effects
@@
 			)
 		)
-		(property "Datasheet" "~"
+		(property "Datasheet" "https://jlcpcb.com/api/file/downloadByFileSystemAccessId/8603345729432014848"
 			(at 138.43 64.77 0)
 			(effects
@@
 			)
 		)
-		(property "LPN" "C307331"
+		(property "LPN" "C22435929"
 			(at 138.43 64.77 0)
 			(effects
@@
 			)
 		)
-		(property "MPN" "CL05B104KB54PNC"
+		(property "MPN" "CGA0201X7R104K160ET "
 			(at 138.43 64.77 0)
 			(effects
@@
 			)
 		)
-		(property "Footprint" "Capacitor_SMD:C_0402_1005Metric"
+		(property "Footprint" "Capacitor_SMD:C_0201_0603Metric"
 			(at 115.57 64.77 0)
 			(effects
@@
 			)
 		)
-		(property "Datasheet" "~"
+		(property "Datasheet" "https://jlcpcb.com/api/file/downloadByFileSystemAccessId/8603345729432014848"
 			(at 115.57 64.77 0)
 			(effects
@@
 			)
 		)
-		(property "LPN" "C307331"
+		(property "LPN" "C22435929"
 			(at 115.57 64.77 0)
 			(effects
@@
 			)
 		)
-		(property "MPN" "CL05B104KB54PNC"
+		(property "MPN" "CGA0201X7R104K160ET "
 			(at 115.57 64.77 0)
 			(effects
@@
 			)
 		)
-		(property "Footprint" "Capacitor_SMD:C_0402_1005Metric"
+		(property "Footprint" "Capacitor_SMD:C_0201_0603Metric"
 			(at 130.81 64.77 0)
 			(effects
@@
 			)
 		)
-		(property "Datasheet" "~"
+		(property "Datasheet" "https://jlcpcb.com/api/file/downloadByFileSystemAccessId/8603345729432014848"
 			(at 130.81 64.77 0)
 			(effects
@@
 			)
 		)
-		(property "LPN" "C307331"
+		(property "LPN" "C22435929"
 			(at 130.81 64.77 0)
 			(effects
@@
 			)
 		)
-		(property "MPN" "CL05B104KB54PNC"
+		(property "MPN" "CGA0201X7R104K160ET "
 			(at 130.81 64.77 0)
 			(effects
@@
 			)
 		)
-		(property "Footprint" "Capacitor_SMD:C_0402_1005Metric"
+		(property "Footprint" "Capacitor_SMD:C_0201_0603Metric"
 			(at 142.24 128.27 0)
 			(effects
@@
 			)
 		)
-		(property "Datasheet" "~"
+		(property "Datasheet" "https://jlcpcb.com/api/file/downloadByFileSystemAccessId/8603345729432014848"
 			(at 142.24 128.27 0)
 			(effects
@@
 			)
 		)
-		(property "LPN" "C307331"
+		(property "LPN" "C22435929"
 			(at 142.24 128.27 0)
 			(effects
@@
 			)
 		)
-		(property "MPN" "CL05B104KB54PNC"
+		(property "MPN" "CGA0201X7R104K160ET "
 			(at 142.24 128.27 0)
 			(effects

Commit message: [¢arrier] Placed decoupling for some banks, placed dc-dc converterss (next) switch dc-dc converter pins around, switch adc-inputs around
Connections:
- net VAUX: now reaches C310.1, C311.1, C312.1, C313.1, IC1.G11 (VCCAUX_1), IC1.L7 (VCCAUX_2), L301.1
Changed lines of the file:
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@@
+		)
+	)
+	(label "VAUX"
+		(at 142.24 124.46 0)
+		(effects
+			(font
+				(size 1.27 1.27)
+			)
+			(justify left bottom)
 		)
 	)

Commit message: [¢arrier] Placed power supply circuitry appropraitely, changed power connector (next) Place schmitt triggers between usb and power, put critical circuitry closer together, place config circuitry
Connections:
- net VAUX_2V5 renamed +2V5
Changed lines of the file:
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@@
 	(wire
 		(pts
-			(xy 120.65 124.46) (xy 124.46 124.46)
+			(xy 118.11 124.46) (xy 124.46 124.46)
 		)
 		(stroke
@@
 		)
 	)
-	(global_label "VAUX_2V5"
-		(shape passive)
-		(at 120.65 124.46 180)
-		(fields_autoplaced yes)
-		(effects
-			(font
-				(size 1.27 1.27)
-			)
-			(justify right)
-		)
-		(property "Intersheetrefs" "${INTERSHEET_REFS}"
-			(at 109.5837 124.46 0)
-			(effects
-				(font
-					(size 1.27 1.27)
-				)
-				(justify right)
-				(hide yes)
-			)
-		)
-	)
 	(symbol
 		(lib_id "Device:C_Small")
@@
 					(unit 1)
 				)
+			)
+		)
+	)
+	(symbol
+		(lib_id "power:+2V5")
+		(at 118.11 124.46 0)
+		(unit 1)
+		(exclude_from_sim no)
+		(in_bom yes)
+		(on_board yes)
+		(dnp no)
+		(fields_autoplaced yes)
+		(property "Reference" "#PWR0304"
+			(at 118.11 128.27 0)
+			(effects
+				(font
+					(size 1.27 1.27)
+				)
+				(hide yes)
+			)
+		)
+		(property "Value" "+2V5"
+			(at 118.11 119.38 0)
+			(effects
+				(font
+					(size 1.27 1.27)
+				)
+			)
+		)
+		(property "Footprint" ""
+			(at 118.11 124.46 0)
+			(effects
+				(font
+					(size 1.27 1.27)
+				)
+				(hide yes)
+			)
+		)
+		(property "Datasheet" ""
+			(at 118.11 124.46 0)
+			(effects
+				(font
+					(size 1.27 1.27)
+				)
+				(hide yes)
+			)
+		)
+		(property "Description" "Power symbol creates a global label with name \"+2V5\""
+			(at 118.11 124.46 0)
+			(effects
+				(font
+					(size 1.27 1.27)
+				)
+				(hide yes)
+			)
+		)
+		(pin "1"
+		)
+		(instances
+			(project ""
+				(path "/25b015c9-ab13-4427-b72c-b6f348597100/aad6bec2-3cac-4ef0-abf0-8e1f80301155"
+					(reference "#PWR0304")
+					(unit 1)
+				)
